File: schematic/board/lidar_made_by_apple.sch (EAGLE design)
At the start: 90 parts, among them J1 U.FL-R-SMT-1_10_, J2 U.FL-R-SMT-1_10_

Commit message: ага угу
Connections:
- net AGND: now also C1.2, C14.1, C33.2, C4.2, C5.2, D6.P$1, J1.1, J1.2, R14.2, U$5.GND
- net GND: no longer C1.2, C10.1, C11.1, C14.1, C33.2, C4.2, C5.2, D6.P$1, J1.1, J1.2, R14.2, R3.1, U$13.S, U$5.GND
- net PGND: now also C10.1, C11.1, R3.1, U$13.S
Changed lines of the file:
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@@
 <label x="327.66" y="137.16" size="1.778" layer="95"/>
+</segment>
+<segment>
+<pinref part="U$13" gate="G$1" pin="S"/>
+<wire x1="363.22" y1="127" x2="363.22" y2="114.3" width="0.1524" layer="91"/>
+<pinref part="R3" gate="G$1" pin="1"/>
+<wire x1="353.06" y1="116.84" x2="353.06" y2="114.3" width="0.1524" layer="91"/>
+<wire x1="353.06" y1="114.3" x2="363.22" y2="114.3" width="0.1524" layer="91"/>
+<wire x1="363.22" y1="114.3" x2="363.22" y2="109.22" width="0.1524" layer="91"/>
+<junction x="363.22" y="114.3"/>
+<label x="365.76" y="106.68" size="1.778" layer="95" rot="R180"/>
+</segment>
+<segment>
+<pinref part="C10" gate="G$1" pin="1"/>
+<wire x1="401.32" y1="127" x2="401.32" y2="114.3" width="0.1524" layer="91"/>
+<label x="403.86" y="114.3" size="1.778" layer="95" rot="R180"/>
+</segment>
+<segment>
+<pinref part="C11" gate="G$1" pin="1"/>
+<wire x1="424.18" y1="127" x2="424.18" y2="114.3" width="0.1524" layer="91"/>
+<label x="426.72" y="114.3" size="1.778" layer="95" rot="R180"/>
 </segment>
 </net>
@@
 <net name="GND" class="0">
 <segment>
-<pinref part="C4" gate="G$1" pin="2"/>
-<wire x1="134.62" y1="-53.34" x2="134.62" y2="-55.88" width="0.1524" layer="91"/>
-<wire x1="134.62" y1="-55.88" x2="124.46" y2="-55.88" width="0.1524" layer="91"/>
-<pinref part="C1" gate="G$1" pin="2"/>
-<wire x1="124.46" y1="-55.88" x2="124.46" y2="-53.34" width="0.1524" layer="91"/>
-<wire x1="124.46" y1="-55.88" x2="124.46" y2="-58.42" width="0.1524" layer="91"/>
-<junction x="124.46" y="-55.88"/>
-<label x="124.46" y="-58.42" size="1.778" layer="95" rot="R90"/>
-</segment>
-<segment>
-<pinref part="C5" gate="G$1" pin="2"/>
-<wire x1="154.94" y1="-63.5" x2="154.94" y2="-68.58" width="0.1524" layer="91"/>
-<label x="152.4" y="-70.358" size="1.778" layer="95"/>
-</segment>
-<segment>
-<pinref part="U$5" gate="G$1" pin="GND"/>
-<wire x1="187.96" y1="-48.26" x2="193.04" y2="-48.26" width="0.1524" layer="91"/>
-<wire x1="193.04" y1="-48.26" x2="193.04" y2="-45.72" width="0.1524" layer="91"/>
-<label x="190.5" y="-45.72" size="1.778" layer="95"/>
-</segment>
-<segment>
-<pinref part="D6" gate="G$1" pin="P$1"/>
-<wire x1="142.86" y1="-80.74" x2="142.86" y2="-86.36" width="0.1524" layer="91"/>
-<label x="140.208" y="-88.138" size="1.778" layer="95"/>
-</segment>
-<segment>
-<pinref part="C33" gate="G$1" pin="2"/>
-<wire x1="139.7" y1="-93.98" x2="144.78" y2="-93.98" width="0.1524" layer="91"/>
-<label x="142.24" y="-93.98" size="1.778" layer="95"/>
-</segment>
-<segment>
-<pinref part="C14" gate="G$1" pin="1"/>
-<wire x1="241.3" y1="-17.78" x2="246.38" y2="-17.78" width="0.1524" layer="91"/>
-<label x="248.92" y="-20.32" size="1.778" layer="95" rot="R90"/>
-</segment>
-<segment>
-<pinref part="R14" gate="G$1" pin="2"/>
-<wire x1="228.6" y1="-68.58" x2="228.6" y2="-76.2" width="0.1524" layer="91"/>
-<label x="226.06" y="-78.74" size="1.778" layer="95"/>
-</segment>
-<segment>
-<pinref part="J1" gate="G$1" pin="2"/>
-<wire x1="193.04" y1="-78.74" x2="198.12" y2="-78.74" width="0.1524" layer="91"/>
-<label x="195.58" y="-78.74" size="1.778" layer="95"/>
-</segment>
-<segment>
-<pinref part="J1" gate="G$1" pin="1"/>
-<wire x1="172.72" y1="-78.74" x2="167.64" y2="-78.74" width="0.1524" layer="91"/>
-<label x="165.1" y="-78.74" size="1.778" layer="95"/>
-</segment>
-<segment>
 <wire x1="17.78" y1="-27.94" x2="17.78" y2="-25.4" width="0.1524" layer="91"/>
 <pinref part="W1" gate="G$1" pin="2"/>
@@
 <pinref part="C18" gate="G$1" pin="1"/>
 <pinref part="C20" gate="G$1" pin="1"/>
-</segment>
-<segment>
-<pinref part="U$13" gate="G$1" pin="S"/>
-<wire x1="363.22" y1="127" x2="363.22" y2="114.3" width="0.1524" layer="91"/>
-<pinref part="R3" gate="G$1" pin="1"/>
-<wire x1="353.06" y1="116.84" x2="353.06" y2="114.3" width="0.1524" layer="91"/>
-<wire x1="353.06" y1="114.3" x2="363.22" y2="114.3" width="0.1524" layer="91"/>
-<wire x1="363.22" y1="114.3" x2="363.22" y2="109.22" width="0.1524" layer="91"/>
-<junction x="363.22" y="114.3"/>
-<label x="365.76" y="106.68" size="1.778" layer="95" rot="R180"/>
-</segment>
-<segment>
-<pinref part="C10" gate="G$1" pin="1"/>
-<wire x1="401.32" y1="127" x2="401.32" y2="114.3" width="0.1524" layer="91"/>
-<label x="403.86" y="114.3" size="1.778" layer="95" rot="R180"/>
-</segment>
-<segment>
-<pinref part="C11" gate="G$1" pin="1"/>
-<wire x1="424.18" y1="127" x2="424.18" y2="114.3" width="0.1524" layer="91"/>
-<label x="426.72" y="114.3" size="1.778" layer="95" rot="R180"/>
 </segment>
 <segment>
@@
 <label x="25.4" y="-30.48" size="1.778" layer="95"/>
 </segment>
-</net>
+<segment>
+<pinref part="U$5" gate="G$1" pin="GND"/>
+<wire x1="187.96" y1="-48.26" x2="193.04" y2="-48.26" width="0.1524" layer="91"/>
+<wire x1="193.04" y1="-48.26" x2="193.04" y2="-45.72" width="0.1524" layer="91"/>
+<label x="190.5" y="-45.72" size="1.778" layer="95"/>
+</segment>
+<segment>
+<pinref part="C4" gate="G$1" pin="2"/>
+<wire x1="134.62" y1="-53.34" x2="134.62" y2="-55.88" width="0.1524" layer="91"/>
+<wire x1="134.62" y1="-55.88" x2="124.46" y2="-55.88" width="0.1524" layer="91"/>
+<pinref part="C1" gate="G$1" pin="2"/>
+<wire x1="124.46" y1="-55.88" x2="124.46" y2="-53.34" width="0.1524" layer="91"/>
+<wire x1="124.46" y1="-55.88" x2="124.46" y2="-58.42" width="0.1524" layer="91"/>
+<junction x="124.46" y="-55.88"/>
+<label x="124.46" y="-58.42" size="1.778" layer="95" rot="R90"/>
+</segment>
+<segment>
+<pinref part="C33" gate="G$1" pin="2"/>
+<wire x1="139.7" y1="-93.98" x2="144.78" y2="-93.98" width="0.1524" layer="91"/>
+<label x="142.24" y="-93.98" size="1.778" layer="95"/>
+</segment>
+<segment>
+<pinref part="D6" gate="G$1" pin="P$1"/>
+<wire x1="142.86" y1="-80.74" x2="142.86" y2="-86.36" width="0.1524" layer="91"/>
+<label x="140.208" y="-88.138" size="1.778" layer="95"/>
+</segment>
+<segment>
+<pinref part="C5" gate="G$1" pin="2"/>
+<wire x1="154.94" y1="-63.5" x2="154.94" y2="-68.58" width="0.1524" layer="91"/>
+<label x="152.4" y="-70.358" size="1.778" layer="95"/>
+</segment>
+<segment>
+<pinref part="J1" gate="G$1" pin="1"/>
+<wire x1="172.72" y1="-78.74" x2="167.64" y2="-78.74" width="0.1524" layer="91"/>
+<label x="165.1" y="-78.74" size="1.778" layer="95"/>
+</segment>
+<segment>
+<pinref part="R14" gate="G$1" pin="2"/>
+<wire x1="228.6" y1="-68.58" x2="228.6" y2="-76.2" width="0.1524" layer="91"/>
+<label x="226.06" y="-78.74" size="1.778" layer="95"/>
+</segment>
+<segment>
+<pinref part="C14" gate="G$1" pin="1"/>
+<wire x1="241.3" y1="-17.78" x2="246.38" y2="-17.78" width="0.1524" layer="91"/>
+<label x="248.92" y="-20.32" size="1.778" layer="95" rot="R90"/>
+</segment>
+<segment>
+<pinref part="J1" gate="G$1" pin="2"/>
+<wire x1="193.04" y1="-78.74" x2="198.12" y2="-78.74" width="0.1524" layer="91"/>
+<label x="195.58" y="-78.74" size="1.778" layer="95"/>
+</segment>
+</net>

Commit message: Безумие — это точное повторение одного и того же действия раз за разом в надежде на изменение
Connections:
- net 3V3: no longer L1.1, R31.2, U$10.EN_STOP1, U$10.EN_STOP2
- net 3V3_REF: now also L1.1
- net V_TDC: now also R31.2, U$10.EN_STOP1, U$10.EN_STOP2
Changed lines of the file:
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@@
 <net name="3V3" class="0">
-<segment>
-<pinref part="R31" gate="G$1" pin="2"/>
-<wire x1="114.3" y1="144.78" x2="114.3" y2="147.32" width="0.1524" layer="91"/>
-<label x="109.22" y="147.32" size="1.778" layer="95"/>
-</segment>
 <segment>
 <label x="139.7" y="203.2" size="1.778" layer="95"/>
 <pinref part="L9" gate="G$1" pin="2"/>
 <wire x1="137.16" y1="203.2" x2="144.78" y2="203.2" width="0.1524" layer="91"/>
-</segment>
-<segment>
-<pinref part="U$10" gate="G$1" pin="EN_STOP2"/>
-<wire x1="177.8" y1="147.32" x2="182.88" y2="147.32" width="0.1524" layer="91"/>
-<pinref part="U$10" gate="G$1" pin="EN_STOP1"/>
-<wire x1="182.88" y1="147.32" x2="195.58" y2="147.32" width="0.1524" layer="91"/>
-<wire x1="177.8" y1="152.4" x2="182.88" y2="152.4" width="0.1524" layer="91"/>
-<wire x1="182.88" y1="152.4" x2="182.88" y2="147.32" width="0.1524" layer="91"/>
-<junction x="182.88" y="147.32"/>
-<label x="187.96" y="147.32" size="1.778" layer="95"/>
-</segment>
-<segment>
-<wire x1="124.46" y1="-25.4" x2="124.46" y2="-20.32" width="0.1524" layer="91"/>
-<label x="121.92" y="-20.32" size="1.778" layer="95"/>
-<pinref part="L1" gate="G$1" pin="1"/>
 </segment>
 <segment>
@@
 <label x="12.7" y="-119.38" size="1.778" layer="95" rot="R90"/>
 <pinref part="U$4" gate="G$1" pin="VCCI/VCCO"/>
+</segment>
+<segment>
+<wire x1="124.46" y1="-25.4" x2="124.46" y2="-20.32" width="0.1524" layer="91"/>
+<label x="121.92" y="-20.32" size="1.778" layer="95"/>
+<pinref part="L1" gate="G$1" pin="1"/>
 </segment>
 </net>
@@
 <wire x1="116.84" y1="203.2" x2="116.84" y2="180.34" width="0.1524" layer="91"/>
 </segment>
-</net>
+<segment>
+<pinref part="U$10" gate="G$1" pin="EN_STOP2"/>
+<wire x1="177.8" y1="147.32" x2="182.88" y2="147.32" width="0.1524" layer="91"/>
+<pinref part="U$10" gate="G$1" pin="EN_STOP1"/>
+<wire x1="182.88" y1="147.32" x2="195.58" y2="147.32" width="0.1524" layer="91"/>
+<wire x1="177.8" y1="152.4" x2="182.88" y2="152.4" width="0.1524" layer="91"/>
+<wire x1="182.88" y1="152.4" x2="182.88" y2="147.32" width="0.1524" layer="91"/>
+<junction x="182.88" y="147.32"/>
+<label x="187.96" y="147.32" size="1.778" layer="95"/>
+</segment>
+<segment>
+<pinref part="R31" gate="G$1" pin="2"/>
+<wire x1="114.3" y1="144.78" x2="114.3" y2="147.32" width="0.1524" layer="91"/>
+<label x="109.22" y="147.32" size="1.778" layer="95"/>
+</segment>
+</net>

Commit message: Даниил на протяжении 510 лет переделывает плату лидара
Connections:
- net 5V: now also U$12.IN
- net V_BAT: no longer U$12.IN
Changed lines of the file:
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@@
-</segment>
-<segment>
-<pinref part="U$12" gate="G$1" pin="IN"/>
-<wire x1="38.1" y1="-48.26" x2="33.02" y2="-48.26" width="0.1524" layer="91"/>
-<label x="30.48" y="-48.26" size="1.778" layer="95"/>
 </segment>
 <segment>
@@
 <label x="314.96" y="63.5" size="1.778" layer="95"/>
 </segment>
+<segment>
+<pinref part="U$12" gate="G$1" pin="IN"/>
+<wire x1="38.1" y1="-48.26" x2="33.02" y2="-48.26" width="0.1524" layer="91"/>
+<label x="30.48" y="-48.26" size="1.778" layer="95"/>
+</segment>
 </net>

Commit message: почти добавил новый разъём
Parts:
- removed JP3: (no value), pinhead:PINHD-1X15
- removed JP4, JP5: (no value), pinhead:PINHD-1X9
- added U$15, U$16: PBS_SMD_X9, NEON-BLADE-2024:PBS_SMD_X9
- added U$17: PBS_SMD_X15, NEON-BLADE-2024:PBS_SMD_X15
Connections:
- net 1MISO: now also U$17.3; no longer JP3.3
- net 1MOSI: now also U$17.2; no longer JP3.2
- net 1SCK: now also U$17.1; no longer JP3.1
- net 3V3: now also U$17.5; no longer JP3.5
- net 4MISO: now also U$15.4; no longer JP5.4
- net 4MOSI: now also U$15.3; no longer JP5.3
- net 4SCK: now also U$15.2; no longer JP5.2
- net 5MISO: now also U$17.11; no longer JP3.11
- net 5MOSI: now also U$17.10; no longer JP3.10
- net 5SCK: now also U$17.9; no longer JP3.9
- net 5V: now also U$16.1; no longer JP4.1
- net APD_FB_VOLT: now also U$15.8; no longer JP5.8
- net APD_PWM: now also U$15.9; no longer JP5.9
- net CE_NRF: now also U$17.7; no longer JP3.7
- net CS_LIS: now also U$17.4; no longer JP3.4
- net CS_LSM: now also U$17.12; no longer JP3.12
- net CS_NRF: now also U$17.8; no longer JP3.8
- net CS_TDC: now also U$15.5; no longer JP5.5
- net GND: now also U$17.6; no longer JP3.6
- net LASER_COMP: now also U$15.6; no longer JP5.6
- net N$28: now also U$17.13; no longer JP3.13
- net N$30: now also U$17.15; no longer JP3.15
- net SCL: now also U$16.9; no longer JP4.9
- net SDA: now also U$16.8; no longer JP4.8
- net SDIO_CK: now also U$16.5; no longer JP4.5
- net SDIO_CMD: now also U$16.4; no longer JP4.4
- net SDIO_DAT0: now also U$16.6; no longer JP4.6
- net SDIO_DAT1: now also U$16.7; no longer JP4.7
- net SDIO_DAT2: now also U$16.2; no longer JP4.2
- net SDIO_DAT3: now also U$16.3; no longer JP4.3
- net TDC_INT: now also U$15.7; no longer JP5.7
- net USIL_ON: now also U$15.1; no longer JP5.1
- net V_BAT: now also U$17.14; no longer JP3.14

Commit message: переделки по плате
Connections:
- removed net 1MISO: U$17.3
- removed net 1MOSI: U$17.2
- removed net 1SCK: U$17.1
- removed net 5MISO: U$17.11
- removed net 5MOSI: U$17.10
- removed net 5SCK: U$17.9
- removed net CE_NRF: U$17.7
- removed net CS_LIS: U$17.4
- removed net CS_LSM: U$17.12
- removed net CS_NRF: U$17.8
- removed net N$30: U$17.15
- removed net SCL: U$16.9
- removed net SDA: U$16.8
- removed net SDIO_CK: U$16.5
- removed net SDIO_CMD: U$16.4
- removed net SDIO_DAT0: U$16.6
- removed net SDIO_DAT1: U$16.7
- removed net SDIO_DAT2: U$16.2
- removed net SDIO_DAT3: U$16.3
- removed net USIL_ON: U$15.1
- net 3V3: now also L1.1
- net 3V3_REF: no longer L1.1
- net COMP_DAC: now also U$17.13
- net GND: no longer C20.1
- net N$28: now also C20.1; no longer U$17.13
Other:
- moved on the sheet: C18, C20
