File: schematic/board/lidar_made_by_apple.sch (EAGLE design)
At the start: 88 parts, among them J1 U.FL-R-SMT-1_10_, J2 U.FL-R-SMT-1_10_

Commit message: добавил полигоны на плату и добавил буквы на разъём
Changed lines of the file:
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@@
 <grid distance="0.1" unitdist="inch" unit="inch" style="lines" multiple="1" display="no" altdistance="0.01" altunitdist="inch" altunit="inch"/>
 <layers>
-<layer number="1" name="Top" color="4" fill="1" visible="yes" active="no"/>
-<layer number="16" name="Bottom" color="1" fill="1" visible="yes" active="no"/>
-<layer number="17" name="Pads" color="2" fill="1" visible="yes" active="no"/>
-<layer number="18" name="Vias" color="2" fill="1" visible="yes" active="no"/>
-<layer number="19" name="Unrouted" color="6" fill="1" visible="yes" active="no"/>
-<layer number="20" name="Dimension" color="24" fill="1" visible="yes" active="no"/>
-<layer number="21" name="tPlace" color="7" fill="1" visible="yes" active="no"/>
-<layer number="22" name="bPlace" color="7" fill="1" visible="yes" active="no"/>
-<layer number="23" name="tOrigins" color="15" fill="1" visible="yes" active="no"/>
-<layer number="24" name="bOrigins" color="15" fill="1" visible="yes" active="no"/>
-<layer number="25" name="tNames" color="7" fill="1" visible="yes" active="no"/>
-<layer number="26" name="bNames" color="7" fill="1" visible="yes" active="no"/>
-<layer number="27" name="tValues" color="7" fill="1" visible="yes" active="no"/>
-<layer number="28" name="bValues" color="7" fill="1" visible="yes" active="no"/>
+<layer number="1" name="Top" color="4" fill="1" visible="no" active="no"/>
+<layer number="16" name="Bottom" color="1" fill="1" visible="no" active="no"/>
+<layer number="17" name="Pads" color="2" fill="1" visible="no" active="no"/>
+<layer number="18" name="Vias" color="2" fill="1" visible="no" active="no"/>
+<layer number="19" name="Unrouted" color="6" fill="1" visible="no" active="no"/>
+<layer number="20" name="Dimension" color="24" fill="1" visible="no" active="no"/>
+<layer number="21" name="tPlace" color="7" fill="1" visible="no" active="no"/>
+<layer number="22" name="bPlace" color="7" fill="1" visible="no" active="no"/>
+<layer number="23" name="tOrigins" color="15" fill="1" visible="no" active="no"/>
+<layer number="24" name="bOrigins" color="15" fill="1" visible="no" active="no"/>
+<layer number="25" name="tNames" color="7" fill="1" visible="no" active="no"/>
+<layer number="26" name="bNames" color="7" fill="1" visible="no" active="no"/>
+<layer number="27" name="tValues" color="7" fill="1" visible="no" active="no"/>
+<layer number="28" name="bValues" color="7" fill="1" visible="no" active="no"/>
 <layer number="29" name="tStop" color="7" fill="3" visible="no" active="no"/>
 <layer number="30" name="bStop" color="7" fill="6" visible="no" active="no"/>
@@
 <layer number="35" name="tGlue" color="7" fill="4" visible="no" active="no"/>
 <layer number="36" name="bGlue" color="7" fill="5" visible="no" active="no"/>
-<layer number="37" name="tTest" color="7" fill="1" visible="yes" active="no"/>
-<layer number="38" name="bTest" color="7" fill="1" visible="yes" active="no"/>
+<layer number="37" name="tTest" color="7" fill="1" visible="no" active="no"/>
+<layer number="38" name="bTest" color="7" fill="1" visible="no" active="no"/>
 <layer number="39" name="tKeepout" color="4" fill="11" visible="no" active="no"/>
 <layer number="40" name="bKeepout" color="1" fill="11" visible="no" active="no"/>
@@
 <layer number="44" name="Drills" color="7" fill="1" visible="no" active="no"/>
 <layer number="45" name="Holes" color="7" fill="1" visible="no" active="no"/>
-<layer number="46" name="Milling" color="3" fill="1" visible="yes" active="no"/>
-<layer number="47" name="Measures" color="7" fill="1" visible="yes" active="no"/>
-<layer number="48" name="Document" color="7" fill="1" visible="yes" active="no"/>
-<layer number="49" name="Reference" color="7" fill="1" visible="yes" active="no"/>
-<layer number="50" name="dxf" color="7" fill="1" visible="yes" active="no"/>
-<layer number="51" name="tDocu" color="7" fill="1" visible="yes" active="no"/>
-<layer number="52" name="bDocu" color="7" fill="1" visible="yes" active="no"/>
-<layer number="53" name="tGND_GNDA" color="7" fill="9" visible="yes" active="no"/>
-<layer number="54" name="bGND_GNDA" color="1" fill="9" visible="yes" active="no"/>
-<layer number="56" name="wert" color="7" fill="1" visible="yes" active="no"/>
-<layer number="57" name="tCAD" color="7" fill="1" visible="yes" active="no"/>
-<layer number="59" name="tCarbon" color="7" fill="1" visible="yes" active="no"/>
-<layer number="60" name="bCarbon" color="7" fill="1" visible="yes" active="no"/>
+<layer number="46" name="Milling" color="3" fill="1" visible="no" active="no"/>
+<layer number="47" name="Measures" color="7" fill="1" visible="no" active="no"/>
+<layer number="48" name="Document" color="7" fill="1" visible="no" active="no"/>
+<layer number="49" name="Reference" color="7" fill="1" visible="no" active="no"/>
+<layer number="50" name="dxf" color="7" fill="1" visible="no" active="no"/>
+<layer number="51" name="tDocu" color="7" fill="1" visible="no" active="no"/>
+<layer number="52" name="bDocu" color="7" fill="1" visible="no" active="no"/>
+<layer number="53" name="tGND_GNDA" color="7" fill="9" visible="no" active="no"/>
+<layer number="54" name="bGND_GNDA" color="1" fill="9" visible="no" active="no"/>
+<layer number="56" name="wert" color="7" fill="1" visible="no" active="no"/>
+<layer number="57" name="tCAD" color="7" fill="1" visible="no" active="no"/>
+<layer number="59" name="tCarbon" color="7" fill="1" visible="no" active="no"/>
+<layer number="60" name="bCarbon" color="7" fill="1" visible="no" active="no"/>
 <layer number="88" name="SimResults" color="9" fill="1" visible="yes" active="yes"/>
 <layer number="89" name="SimProbes" color="9" fill="1" visible="yes" active="yes"/>
@@
 <segment>
 <pinref part="U$10" gate="G$1" pin="MOSI"/>
-<wire x1="142.24" y1="132.08" x2="132.08" y2="132.08" width="0.1524" layer="91"/>
-<label x="132.08" y="132.08" size="1.778" layer="95"/>
+<wire x1="142.24" y1="132.08" x2="129.54" y2="132.08" width="0.1524" layer="91"/>
+<label x="129.54" y="132.08" size="1.778" layer="95"/>
 </segment>
 <segment>
@@
 <segment>
 <pinref part="U$10" gate="G$1" pin="MISO"/>
-<wire x1="142.24" y1="127" x2="132.08" y2="127" width="0.1524" layer="91"/>
-<label x="132.08" y="127" size="1.778" layer="95"/>
+<wire x1="142.24" y1="127" x2="129.54" y2="127" width="0.1524" layer="91"/>
+<label x="129.54" y="127" size="1.778" layer="95"/>
 </segment>
 <segment>
@@
 <segment>
 <pinref part="U$10" gate="G$1" pin="SSN"/>
-<wire x1="142.24" y1="142.24" x2="132.08" y2="142.24" width="0.1524" layer="91"/>
-<label x="132.08" y="142.24" size="1.778" layer="95"/>
+<wire x1="142.24" y1="142.24" x2="129.54" y2="142.24" width="0.1524" layer="91"/>
+<label x="129.54" y="142.24" size="1.778" layer="95"/>
 </segment>
 <segment>
@@
 <segment>
 <pinref part="U$10" gate="G$1" pin="SCK"/>
-<wire x1="142.24" y1="137.16" x2="132.08" y2="137.16" width="0.1524" layer="91"/>
-<label x="132.08" y="137.16" size="1.778" layer="95"/>
-</segment>
-<segment>
+<wire x1="142.24" y1="137.16" x2="129.54" y2="137.16" width="0.1524" layer="91"/>
+<label x="129.54" y="137.16" size="1.778" layer="95"/>
+</segment>
+<segment>

Commit message: забыи отладочные пины...
Parts:
- C18: value 22F -> 22uF
- C19, C2, C9: device rcl:C-EUC1210 -> rcl:C-EUC1206
Connections:
- net TDC_INT: no longer U$15.7
Changed lines of the file:
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@@
 <part name="C22" library="rcl" library_urn="urn:adsk.eagle:library:334" deviceset="C-EU" device="C0603" package3d_urn="urn:adsk.eagle:package:23616/2" value="10pF"/>
 <part name="L9" library="NEON-BLADE-2024" deviceset="L_BEAD" device=""/>
-<part name="C18" library="rcl" library_urn="urn:adsk.eagle:library:334" deviceset="C-EU" device="C1210" package3d_urn="urn:adsk.eagle:package:23619/2" value="22F"/>
+<part name="C18" library="rcl" library_urn="urn:adsk.eagle:library:334" deviceset="C-EU" device="C1210" package3d_urn="urn:adsk.eagle:package:23619/2" value="22uF"/>
 <part name="C20" library="rcl" library_urn="urn:adsk.eagle:library:334" deviceset="C-EU" device="C1210" package3d_urn="urn:adsk.eagle:package:23619/2" value="22uF"/>
 <part name="U$9" library="NEON-BLADE-2024" deviceset="C005R" device=""/>
@@
 <part name="L3" library="NEON-BLADE-2024" deviceset="L_10MKH" device=""/>
 <part name="L2" library="NEON-BLADE-2024" deviceset="L_BEAD" device=""/>
-<part name="C2" library="rcl" library_urn="urn:adsk.eagle:library:334" deviceset="C-EU" device="C1210" package3d_urn="urn:adsk.eagle:package:23619/2" value="10uF"/>
-<part name="C9" library="rcl" library_urn="urn:adsk.eagle:library:334" deviceset="C-EU" device="C1210" package3d_urn="urn:adsk.eagle:package:23619/2" value="10uF"/>
+<part name="C2" library="rcl" library_urn="urn:adsk.eagle:library:334" deviceset="C-EU" device="C1206" package3d_urn="urn:adsk.eagle:package:23618/2" value="10uF"/>
+<part name="C9" library="rcl" library_urn="urn:adsk.eagle:library:334" deviceset="C-EU" device="C1206" package3d_urn="urn:adsk.eagle:package:23618/2" value="10uF"/>
 <part name="VR1" library="NEON-BLADE-2024" deviceset="3362P-1-502LF" device=""/>
 <part name="U$13" library="NEON-BLADE-2024" deviceset="BSS131" device=""/>
@@
 <part name="U$4" library="NEON-BLADE-2024" deviceset="ADCMP600" device=""/>
 <part name="L10" library="NEON-BLADE-2024" deviceset="L_BEAD" device=""/>
-<part name="C19" library="rcl" library_urn="urn:adsk.eagle:library:334" deviceset="C-EU" device="C1210" package3d_urn="urn:adsk.eagle:package:23619/2" value="10uF"/>
+<part name="C19" library="rcl" library_urn="urn:adsk.eagle:library:334" deviceset="C-EU" device="C1206" package3d_urn="urn:adsk.eagle:package:23618/2" value="10uF"/>
 <part name="U$12" library="NEON-BLADE-2024" deviceset="REF3033" device=""/>
 <part name="VR2" library="NEON-BLADE-2024" deviceset="3362P-1-502LF" device=""/>
@@
 <label x="129.54" y="147.32" size="1.778" layer="95"/>
 </segment>
-<segment>
-<wire x1="434.34" y1="119.38" x2="416.56" y2="119.38" width="0.1524" layer="91"/>
-<label x="416.56" y="119.38" size="1.778" layer="95"/>
-<pinref part="U$15" gate="G$1" pin="7"/>
-</segment>
 </net>

Commit message: Убрал дырку и 100501 раз изменил плату лидара
Parts:
- added U$18, U$19: (no value), NEON-BLADE-2024:VIAS-CONNECT
- C10, C11: value 10nF -> 10nF 250v
- C16, C18, C20: device rcl:C-EUC1210 -> rcl:C-EUC1206
- C17: value 20nF -> 20nF low esr
- R2: value 47 -> 100R
Connections:
- new net APD_V_: R1.2, U$18.2
- new net VLASER_: L8.1, R18.2, U$19.2
- net APD_V: now also U$18.1; no longer R1.2
- net VLASER: now also U$19.1; no longer L8.1, R18.2

Commit message: Считаем, что платы готовы к производству
Parts:
- C10, C33: device rcl:C-EUC0603 -> rcl:C-EUC0805
- C11: value 10nF 250v -> 10nF 250V; device rcl:C-EUC0603 -> rcl:C-EUC0805
- C15, C29: value 100nf -> 100nF
- C17: value 20nF low esr -> 22nF low ESR
- C8: value 100pf -> 100pF
- L3: value L_10MKH -> 10uH
- R15: value 150 -> 150R
- R19: value 0.1 -> R100; device rcl:R-EU_R0603 -> rcl:R-EU_R2512
- R20, R7: value 47 -> 47R
- R27: value 0 -> 0R
- renumbered U$12 to REF3033
Connections:
- removed net N$34: C8.1, R9.1
- removed net TDC_INT: U$10.INT
- net PGND: now also C8.1, R9.1
Other:
- moved on the sheet: R10, R8, R9, U$17

Commit message: переделал плату лидара(((((
Parts:
- removed U$1: UCC27511DBVR, NEON-BLADE-2024:UCC27511DBVR
- added U$12: LM5114, NEON-BLADE-2024:LM5114
- L3: device NEON-BLADE-2024:L_10MKH -> NEON-BLADE-2024:L_15MKH
Connections:
- net LASER_PULSE: now also U$12.IN; no longer U$1.IN+
- net N$1: now also U$12.N_OUT, U$12.P_OUT; no longer U$1.OUTH, U$1.OUTL
- net N$2: now also U$12.VDD; no longer U$1.VDD
- net PGND: now also U$12.INB, U$12.VSS; no longer U$1.GND, U$1.IN-
Changed lines of the file:
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@@
 <?xml version="1.0" encoding="utf-8"?>
 <!DOCTYPE eagle SYSTEM "eagle.dtd">
-<eagle version="9.4.2">
+<eagle version="9.6.2">
 <drawing>
 <settings>
-<setting alwaysvectorfont="yes"/>
+<setting alwaysvectorfont="no"/>
 <setting verticaltext="up"/>
 </settings>
@@
 <part name="R5" library="rcl" library_urn="urn:adsk.eagle:library:334" deviceset="R-EU_" device="R0603" package3d_urn="urn:adsk.eagle:package:23555/3" value="47k"/>
 <part name="R6" library="rcl" library_urn="urn:adsk.eagle:library:334" deviceset="R-EU_" device="R0603" package3d_urn="urn:adsk.eagle:package:23555/3" value="4.7k"/>
-<part name="L3" library="NEON-BLADE-2024" deviceset="L_10MKH" device="" value="10uH"/>
+<part name="L3" library="NEON-BLADE-2024" deviceset="L_15MKH" device="" value="10uH"/>
 <part name="L2" library="NEON-BLADE-2024" deviceset="L_BEAD" device=""/>
 <part name="C2" library="rcl" library_urn="urn:adsk.eagle:library:334" deviceset="C-EU" device="C1206" package3d_urn="urn:adsk.eagle:package:23618/2" value="10uF"/>
@@
 <part name="U$16" library="NEON-BLADE-2024" deviceset="PBS_SMD_X9" device=""/>
 <part name="U$17" library="NEON-BLADE-2024" deviceset="PBS_SMD_X15" device=""/>
-<part name="U$1" library="NEON-BLADE-2024" deviceset="UCC27511DBVR" device=""/>
 <part name="R16" library="rcl" library_urn="urn:adsk.eagle:library:334" deviceset="R-EU_" device="R0603" package3d_urn="urn:adsk.eagle:package:23555/3" value="1k"/>
 <part name="R18" library="rcl" library_urn="urn:adsk.eagle:library:334" deviceset="R-EU_" device="R0603" package3d_urn="urn:adsk.eagle:package:23555/3" value="270"/>
@@
 <part name="U$18" library="NEON-BLADE-2024" deviceset="VIAS-CONNECT" device=""/>
 <part name="U$19" library="NEON-BLADE-2024" deviceset="VIAS-CONNECT" device=""/>
+<part name="U$12" library="NEON-BLADE-2024" deviceset="LM5114" device=""/>
 </parts>
 <sheets>
@@
 <attribute name="VALUE" x="384.81" y="93.98" size="1.778" layer="96"/>
 </instance>
-<instance part="U$1" gate="G$1" x="81.28" y="25.4" smashed="yes"/>
 <instance part="R16" gate="G$1" x="58.42" y="20.32" smashed="yes" rot="R90">
 <attribute name="NAME" x="64.262" y="23.6474" size="1.778" layer="95" rot="R180"/>
@@
 <attribute name="VALUE" x="49.53" y="-37.465" size="1.778" layer="96"/>
 </instance>
+<instance part="U$12" gate="G$1" x="81.28" y="30.48" smashed="yes" rot="R180"/>
 </instances>
 <busses>
@@
 </segment>
 <segment>
-<pinref part="U$1" gate="G$1" pin="IN+"/>
-<wire x1="68.58" y1="27.94" x2="58.42" y2="27.94" width="0.1524" layer="91"/>
 <pinref part="R16" gate="G$1" pin="2"/>
 <wire x1="58.42" y1="27.94" x2="58.42" y2="25.4" width="0.1524" layer="91"/>
-<junction x="58.42" y="27.94"/>
 <wire x1="58.42" y1="27.94" x2="50.8" y2="27.94" width="0.1524" layer="91"/>
-<label x="48.26" y="27.94" size="1.778" layer="95"/>
+<label x="43.18" y="25.4" size="1.778" layer="95"/>
+<pinref part="U$12" gate="G$1" pin="IN"/>
+<wire x1="58.42" y1="27.94" x2="68.58" y2="27.94" width="0.1524" layer="91"/>
 </segment>
 </net>
@@
 </segment>
 <segment>
-<pinref part="U$1" gate="G$1" pin="IN-"/>
-<wire x1="68.58" y1="25.4" x2="66.04" y2="25.4" width="0.1524" layer="91"/>
-<wire x1="66.04" y1="25.4" x2="66.04" y2="22.86" width="0.1524" layer="91"/>
-<pinref part="U$1" gate="G$1" pin="GND"/>
-<wire x1="66.04" y1="22.86" x2="66.04" y2="17.78" width="0.1524" layer="91"/>
-<wire x1="68.58" y1="22.86" x2="66.04" y2="22.86" width="0.1524" layer="91"/>
-<junction x="66.04" y="22.86"/>
-<label x="63.754" y="15.494" size="1.778" layer="95"/>
-</segment>
-<segment>
 <wire x1="106.68" y1="38.1" x2="106.68" y2="33.02" width="0.1524" layer="91"/>
 <label x="109.982" y="33.02" size="1.778" layer="95" rot="R180"/>
@@
 <label x="370.84" y="121.92" size="1.778" layer="95"/>
 <pinref part="U$17" gate="G$1" pin="6"/>
+</segment>
+<segment>
+<pinref part="U$12" gate="G$1" pin="VSS"/>
+<wire x1="68.58" y1="33.02" x2="66.04" y2="33.02" width="0.1524" layer="91"/>
+<label x="66.04" y="33.02" size="1.778" layer="95" rot="R180"/>
+</segment>
+<segment>
+<pinref part="U$12" gate="G$1" pin="INB"/>
+<wire x1="68.58" y1="30.48" x2="66.04" y2="30.48" width="0.1524" layer="91"/>
+<label x="66.04" y="30.48" size="1.778" layer="95" rot="R180"/>
 </segment>
 </net>
@@
 </segment>
 </net>
-<net name="N$1" class="0">
-<segment>
-<pinref part="U$1" gate="G$1" pin="OUTL"/>
-<wire x1="93.98" y1="22.86" x2="96.52" y2="22.86" width="0.1524" layer="91"/>
-<wire x1="96.52" y1="22.86" x2="96.52" y2="25.4" width="0.1524" layer="91"/>
-<pinref part="U$1" gate="G$1" pin="OUTH"/>
-<wire x1="93.98" y1="25.4" x2="96.52" y2="25.4" width="0.1524" layer="91"/>
-<wire x1="96.52" y1="25.4" x2="106.68" y2="25.4" width="0.1524" layer="91"/>
-<junction x="96.52" y="25.4"/>
-<pinref part="U$2" gate="G$1" pin="4G"/>
-<wire x1="106.68" y1="25.4" x2="106.68" y2="21.37" width="0.1524" layer="91"/>
-<wire x1="106.68" y1="21.37" x2="116.46" y2="21.37" width="0.1524" layer="91"/>
-</segment>
-</net>
 <net name="N$2" class="0">
 <segment>
-<pinref part="U$1" gate="G$1" pin="VDD"/>
-<wire x1="93.98" y1="27.94" x2="96.52" y2="27.94" width="0.1524" layer="91"/>
-<wire x1="96.52" y1="27.94" x2="96.52" y2="38.1" width="0.1524" layer="91"/>
 <wire x1="96.52" y1="38.1" x2="99.06" y2="38.1" width="0.1524" layer="91"/>
-<junction x="96.52" y="38.1"/>
 <pinref part="L8" gate="G$1" pin="2"/>
 <pinref part="C16" gate="G$1" pin="1"/>
+<pinref part="U$12" gate="G$1" pin="VDD"/>
+<wire x1="96.52" y1="38.1" x2="96.52" y2="27.94" width="0.1524" layer="91"/>
+<wire x1="96.52" y1="27.94" x2="93.98" y2="27.94" width="0.1524" layer="91"/>
+<junction x="96.52" y="38.1"/>
 </segment>
 </net>
@@
 </segment>
 </net>
+<net name="N$1" class="0">
+<segment>
+<pinref part="U$12" gate="G$1" pin="N_OUT"/>
+<pinref part="U$12" gate="G$1" pin="P_OUT"/>
+<wire x1="93.98" y1="33.02" x2="93.98" y2="30.48" width="0.1524" layer="91"/>
+<pinref part="U$2" gate="G$1" pin="4G"/>
+<wire x1="101.6" y1="25.4" x2="106.68" y2="25.4" width="0.1524" layer="91"/>
+<wire x1="106.68" y1="25.4" x2="106.68" y2="21.37" width="0.1524" layer="91"/>
+<wire x1="106.68" y1="21.37" x2="116.46" y2="21.37" width="0.1524" layer="91"/>
+<wire x1="93.98" y1="33.02" x2="101.6" y2="33.02" width="0.1524" layer="91"/>
+<wire x1="101.6" y1="33.02" x2="101.6" y2="25.4" width="0.1524" layer="91"/>
+<junction x="93.98" y="33.02"/>
+</segment>
+</net>
