File: schematic/board/Up_Main_Board.brd (EAGLE design)
At the start: 79.9 x 73.5 mm, 18 parts

Commit message: исправил верхнюю плату
Parts:
- moved U$2 3.30 mm to (50.0, 40.0)
- moved U$6 3.20 mm to (81.0, 44.0)
- moved U$7 3.20 mm to (19.0, 44.0)
Routing:
- net 4MOSI: track 32.8 -> 39.3 mm
- net CS_TDC: track 51.5 -> 57.9 mm
- net SDIO_CMD: track 30.7 -> 36.8 mm
- net 3V3: track 181.7 -> 186.0 mm
- net GPS_TX: track 80.5 -> 77.2 mm
- net GPS_RX: track 82.8 -> 79.5 mm
- net CS_LSM: track 50.1 -> 46.8 mm
- net CS_NRF: track 49.5 -> 46.2 mm
- net 5SCK: track 38.4 -> 35.1 mm
- net 5MISO: track 83.9 -> 80.6 mm
- net LED: track 7.48 -> 10.5 mm
- net CS_LIS: track 62.8 -> 65.8 mm
- net SCL: track 36.9 -> 39.8 mm
- net CE_NRF: track 50.4 -> 53.3 mm
- net 1MOSI: track 52.5 -> 55.3 mm
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