File: schematic/board/Up_Main_Board.brd (EAGLE design)
At the start: 79.9 x 73.5 mm, 27 parts, among them X1 JST-2-K-S, X2 JST-2-K-S, X3 JST-2-K-S, X4 JST-2-K-S

Commit message: Внес поправки
Other:
- board text added: "BUZZ"
- board text added: "IRF7905"
- board text added: "MSS12D01"
- board text added: "SS12D11"
Changed lines of the file:
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@@
 <text x="50" y="78.7" size="1" layer="21" ratio="15" align="bottom-center">Top board [2024] v.1</text>
 <wire x1="58" y1="80.5" x2="42" y2="80.5" width="0.1" layer="21"/>
-<text x="61.8" y="81.3" size="0.8" layer="26" ratio="15" rot="MR180">[NC]</text>
+<text x="61.3" y="81.3" size="0.8" layer="26" ratio="15" rot="MR180">BUZZ</text>
 <text x="66.8" y="81.3" size="0.8" layer="26" ratio="15" rot="MR180">[NC]</text>
 <text x="87.9" y="51.1" size="0.8" layer="26" ratio="15" rot="MR300">APD_FB</text>
@@
 <text x="53.9" y="74.1" size="0.8" layer="26" ratio="15" rot="MR180" align="bottom-center">5V</text>
 <text x="48.7" y="74.1" size="0.8" layer="26" ratio="15" rot="MR180" align="bottom-center">TX</text>
+<text x="60.3" y="19.5" size="0.8" layer="21" ratio="15">IRF7905</text>
+<text x="43.2" y="24.1" size="0.8" layer="21" ratio="15" rot="R90">SS12D11</text>
+<text x="81.4" y="59.6" size="0.8" layer="21" ratio="15" rot="R285">MSS12D01</text>
+<text x="75.1" y="36.9" size="0.8" layer="26" ratio="15" rot="MR300">[NC]</text>
 </plain>
 <attributes>

Commit message: Убрал дырку и 100501 раз изменил плату лидара
Routing:
- net GND: track 224.7 -> 241.7 mm
Other:
- outline, holes or cut-outs redrawn
- board text removed: "SS12D11"
Changed lines of the file:
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@@
 <?xml version="1.0" encoding="utf-8"?>
 <!DOCTYPE eagle SYSTEM "eagle.dtd">
-<eagle version="9.4.2">
+<eagle version="9.6.2">
 <drawing>
 <settings>
-<setting alwaysvectorfont="yes"/>
+<setting alwaysvectorfont="no"/>
 <setting verticaltext="up"/>
 </settings>
@@
 <text x="48.7" y="74.1" size="0.8" layer="26" ratio="15" rot="MR180" align="bottom-center">TX</text>
 <text x="60.3" y="19.5" size="0.8" layer="21" ratio="15">IRF7905</text>
-<text x="43.2" y="24.1" size="0.8" layer="21" ratio="15" rot="R90">SS12D11</text>
 <text x="81.4" y="59.6" size="0.8" layer="21" ratio="15" rot="R285">MSS12D01</text>
 <text x="75.1" y="36.9" size="0.8" layer="26" ratio="15" rot="MR300">[NC]</text>
+<circle x="27.5" y="59.5" radius="2.5" width="0.0001" layer="20"/>
 </plain>
 <attributes>
@@
 <vertex x="8" y="10"/>
 </polygon>
-<wire x1="14.976475" y1="58.092590625" x2="14.976475" y2="57.023525" width="0.2" layer="1"/>
-<wire x1="14.976475" y1="57.023525" x2="15" y2="57" width="0.2" layer="1"/>
-<via x="15" y="57" extent="1-16" drill="0.35"/>
-<wire x1="15" y1="57" x2="20.05" y2="51.95" width="0.2" layer="16"/>
-<wire x1="20.05" y1="51.95" x2="21.23" y2="52.95" width="0.2" layer="16"/>
 <wire x1="70.47" y1="52.95" x2="70.97" y2="53.45" width="0.5" layer="16"/>
 <wire x1="70.97" y1="53.45" x2="77.2848125" y2="59.7648125" width="0.5" layer="16"/>
@@
 <wire x1="46.16" y1="73" x2="63.08" y2="73" width="0.5" layer="1"/>
 <wire x1="63.08" y1="73" x2="64.63" y2="71.45" width="0.5" layer="1"/>
+<wire x1="21.23" y1="71.45" x2="21.4" y2="71.28" width="0.2" layer="1"/>
+<wire x1="17.1116" y1="59.192590625" x2="21.4" y2="63.480990625" width="0.5" layer="1"/>
+<wire x1="21.4" y1="71.28" x2="21.4" y2="63.480990625" width="0.5" layer="1"/>
+<via x="14.660209375" y="56.973634375" extent="1-16" drill="0.35"/>
+<wire x1="14.660209375" y1="56.973634375" x2="14.660209375" y2="55.939790625" width="0.5" layer="16"/>
+<wire x1="17.65" y1="52.95" x2="21.23" y2="52.95" width="0.5" layer="16"/>
+<wire x1="14.660209375" y1="55.939790625" x2="17.65" y2="52.95" width="0.5" layer="16"/>
+<wire x1="17.1116" y1="59.192590625" x2="16.076475" y2="59.192590625" width="0.5" layer="1"/>
+<wire x1="14.976475" y1="58.092590625" x2="16.076475" y2="59.192590625" width="0.5" layer="1"/>
+<wire x1="14.976475" y1="58.092590625" x2="14.976475" y2="57.2899" width="0.5" layer="1"/>
+<wire x1="14.976475" y1="57.2899" x2="14.660209375" y2="56.973634375" width="0.5" layer="1"/>
 </signal>
 <signal name="3V3">
@@
 <wire x1="49.1782" y1="37.4522" x2="49.5" y2="37.774" width="0.2" layer="16"/>
 <wire x1="68.99870625" y1="36.4" x2="69.399234375" y2="36.800528125" width="0.2" layer="1"/>
-<wire x1="55.5030125" y1="36.4" x2="56.0812125" y2="36.9782" width="0.2" layer="1"/>
+<wire x1="55.6030125" y1="36.4" x2="56.1812125" y2="36.9782" width="0.2" layer="1"/>
 <wire x1="58.325025" y1="36.9782" x2="58.903225" y2="36.4" width="0.2" layer="1"/>
-<wire x1="53.9" y1="36.4" x2="55.5030125" y2="36.4" width="0.2" layer="1"/>
-<wire x1="56.0812125" y1="36.9782" x2="58.325025" y2="36.9782" width="0.2" layer="1"/>
+<wire x1="53.9" y1="36.4" x2="55.6030125" y2="36.4" width="0.2" layer="1"/>
+<wire x1="56.1812125" y1="36.9782" x2="58.325025" y2="36.9782" width="0.2" layer="1"/>
 <wire x1="58.903225" y1="36.4" x2="68.99870625" y2="36.4" width="0.2" layer="1"/>
 </signal>

Commit message: теперь точно готовы
Parts:
- moved R4 2.10 mm to (30.1, 28.8)
- moved X1 1.50 mm to (38.0, 26.2)
- moved X3 1.49 mm to (70.3, 25.2)
- moved X2 1.00 mm to (30.0, 26.2)
Routing:
- net DBG_TX: track 19.4 -> 21.7 mm
- net GND: track 241.7 -> 243.5 mm
- net LED: track 5.23 -> 3.70 mm
- net 5V: track 128.2 -> 126.7 mm
- net N$2: track 10.7 -> 12.0 mm
- net N$6: track 3.78 -> 2.81 mm
Other:
- board size 79.9 x 73.5 mm -> 79.8 x 73.5 mm
