File: schematic/board/Down_Main_Board .brd (EAGLE design)
At the start: 79.9 x 73.5 mm, 23 parts, among them J1 MCX-J-P-H-ST-TH1, J2 U.FL-R-SMT-1_10_

Commit message: почти добавил новый разъём
Parts:
- removed R1, R3: 3k3, rcl:R0603
- removed U$2: BUZZERS8R6, NEON-BLADE-2023:BUZZER-S8R12
- removed U$3: SI2302CDS, NEON-BLADE-2023:SOT23-3
- added BUZZER: BUZZERS8R6, NEON-BLADE-2023:BUZZER-S8R12
- added R30: 100R, rcl:R0603
- added R31: 10k, rcl:R0603
- added SI2301: MOSFET-N, NEON-BLADE-2023:SOT23-3
Connections:
- removed net N$2: R1.1, R3.1, U$3.1
- new net N$20: BUZZER.P$2, SI2301.3
- net 5V: now also BUZZER.P$1; no longer U$2.P$1
- net BUZZER: now also R30.1; no longer R3.2
- net GND: now also R31.2, SI2301.2; no longer R1.2, U$3.2
- net N$1: now also R30.2, R31.1, SI2301.1; no longer U$2.P$2, U$3.3
Routing:
- net BUZZER: track 85.9 -> 74.7 mm
- net SDIO_DAT1: track 59.4 -> 48.6 mm, vias 4 -> 3
- net N$20: track 0.00 -> 8.28 mm
- net N$1: track 12.2 -> 4.34 mm
- net N$2: track 4.76 -> 0.00 mm
- net 5V: track 61.6 -> 58.9 mm

Commit message: переделки по плате
Parts:
- removed JP1, JP2: (no value), pinhead:1X09
- removed JP3: (no value), pinhead:1X15
- added U$2, U$3, U$6, U$7: PBS_SMD_X9, NEON-BLADE-2024:PBS_SMD_X9
- added U$4, U$8: PBS_SMD_X15, NEON-BLADE-2024:PBD_SMD_X15
Connections:
- new net N$2: U$4.14
- new net N$3: U$4.15
- net 1MISO: now also U$4.3, U$8.3; no longer JP3.3
- net 1MOSI: now also U$4.2, U$8.2; no longer JP3.2
- net 1SCK: now also U$4.1, U$8.1; no longer JP3.1
- net 3V3: now also U$4.5, U$8.5; no longer JP3.5
- net 5MISO: now also U$4.11, U$8.11; no longer JP3.11
- net 5MOSI: now also U$4.10, U$8.10; no longer JP3.10
- net 5SCK: now also U$4.9, U$8.9; no longer JP3.9
- net 5V: now also U$2.1, U$6.1; no longer JP1.1
- net BUZZER: now also U$4.13, U$8.13; no longer JP3.13
- net CE_NRF: now also U$4.7, U$8.7; no longer JP3.7
- net CS_LIS: now also U$4.4, U$8.4; no longer JP3.4
- net CS_LSM: now also U$4.12, U$8.12; no longer JP3.12
- net CS_NRF: now also U$4.8, U$8.8; no longer JP3.8
- net GND: now also U$4.6, U$8.6; no longer JP3.6
- net N$12: now also U$8.14; no longer JP3.14
- net N$13: now also U$8.15; no longer JP3.15
- net SCL: now also U$2.9, U$6.9; no longer JP1.9
- net SDA: now also U$2.8, U$6.8; no longer JP1.8
- net SDIO_CK: now also U$2.5, U$6.5; no longer JP1.5
- net SDIO_CMD: now also U$2.4, U$6.4; no longer JP1.4
- net SDIO_DAT0: now also U$2.6, U$6.6; no longer JP1.6
- net SDIO_DAT1: now also U$2.7, U$6.7; no longer JP1.7
- net SDIO_DAT2: now also U$2.2, U$6.2; no longer JP1.2
- net SDIO_DAT3: now also U$2.3, U$6.3; no longer JP1.3
- net USIL_ON: now also U$3.1, U$7.1; no longer JP2.1
Routing:
- net 1SCK: track 73.7 -> 18.5 mm
- net 1MOSI: track 65.8 -> 11.0 mm
- net 1MISO: track 48.0 -> 18.4 mm
- net CS_LIS: track 19.9 -> 0.93 mm
- net 5MISO: track 19.2 -> 0.65 mm
- net 5MOSI: track 16.8 -> 0.63 mm
- net 3V3: track 136.0 -> 120.2 mm, vias 4 -> 3
- net 5SCK: track 14.5 -> 0.62 mm
- net CS_LSM: track 13.8 -> 2.09 mm
- net CS_NRF: track 12.2 -> 0.62 mm
- net CE_NRF: track 9.99 -> 2.03 mm
- net GND: track 222.3 -> 215.6 mm
- net BUZZER: track 74.7 -> 68.3 mm
- net SDIO_CK: track 47.2 -> 46.1 mm

Commit message: ПЕРЕДЕЛАЙ ПАЛТЫ
Other:
- outline, holes or cut-outs redrawn
Changed lines of the file:
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@@
 <board>
 <plain>
-<wire x1="89.9406" y1="52.179140625" x2="79.71443125" y2="76.777840625" width="0.001" layer="20" curve="38.901382"/>
-<wire x1="10.0594" y1="52.179140625" x2="31.55733125" y2="14.94365" width="0.001" layer="20"/>
-<wire x1="75.794009375" y1="75.35091875" x2="79.71443125" y2="76.777840625" width="0.001" layer="20"/>
+<wire x1="25.751290625" y1="25" x2="10.0594" y2="52.179140625" width="0.001" layer="20"/>
+<wire x1="34.98128125" y1="25" x2="25.751290625" y2="25" width="0.001" layer="20"/>
+<wire x1="79.71443125" y1="76.777840625" x2="75.794009375" y2="75.35091875" width="0.001" layer="20"/>
+<wire x1="65.56791875" y1="17.355859375" x2="68.44266875" y2="14.94365" width="0.001" layer="20"/>
 <wire x1="28.86165" y1="83.5" x2="29.5133" y2="79.80428125" width="0.001" layer="20"/>
-<wire x1="41.66693125" y1="10.87763125" x2="40.94246875" y2="14.98626875" width="0.001" layer="20"/>
-<wire x1="68.44266875" y1="14.94365" x2="65.56791875" y2="17.355859375" width="0.001" layer="20"/>
+<wire x1="39.90531875" y1="20.868240625" x2="41.66693125" y2="10.87763125" width="0.001" layer="20"/>
 <wire x1="71.13835" y1="83.5" x2="70.4867" y2="79.80428125" width="0.001" layer="20"/>
-<wire x1="59.05753125" y1="14.98626875" x2="58.33306875" y2="10.87763125" width="0.001" layer="20"/>
-<wire x1="34.43208125" y1="17.355859375" x2="31.55733125" y2="14.94365" width="0.001" layer="20"/>
-<wire x1="20.28556875" y1="76.777840625" x2="24.205990625" y2="75.35091875" width="0.001" layer="20"/>
-<wire x1="68.44266875" y1="14.94365" x2="89.9406" y2="52.179140625" width="0.001" layer="20"/>
-<wire x1="71.13835" y1="83.5" x2="28.86165" y2="83.5" width="0.001" layer="20"/>
+<wire x1="58.33306875" y1="10.87763125" x2="59.05753125" y2="14.98626875" width="0.001" layer="20"/>
+<wire x1="24.205990625" y1="75.35091875" x2="20.28556875" y2="76.777840625" width="0.001" layer="20"/>
+<wire x1="89.9406" y1="52.179140625" x2="68.44266875" y2="14.94365" width="0.001" layer="20"/>
+<wire x1="28.86165" y1="83.5" x2="71.13835" y2="83.5" width="0.001" layer="20"/>
 <wire x1="41.66693125" y1="10.87763125" x2="58.33306875" y2="10.87763125" width="0.001" layer="20" curve="24.048625"/>
+<wire x1="20.28556875" y1="76.777840625" x2="10.0594" y2="52.179140625" width="0.001" layer="20" curve="38.901385"/>
 <wire x1="89.9406" y1="52.179140625" x2="79.71443125" y2="76.777840625" width="0.001" layer="20" curve="38.901385"/>
-<wire x1="20.28556875" y1="76.777840625" x2="10.0594" y2="52.179140625" width="0.001" layer="20" curve="38.901385"/>
+<wire x1="39.90531875" y1="20.868240625" x2="34.98128125" y2="25.000003125" width="0.001" layer="20" curve="79.999971"/>
+<wire x1="65.56791875" y1="17.355859375" x2="59.057534375" y2="14.98626875" width="0.001" layer="20" curve="120.000001"/>
 <wire x1="70.4867" y1="79.80428125" x2="75.79400625" y2="75.350921875" width="0.001" layer="20" curve="120.000013"/>
-<wire x1="65.56791875" y1="17.355859375" x2="59.057534375" y2="14.98626875" width="0.001" layer="20" curve="120.000001"/>
-<wire x1="40.94246875" y1="14.98626875" x2="34.43208125" y2="17.355859375" width="0.001" layer="20" curve="120.000035"/>
 <wire x1="24.205990625" y1="75.35091875" x2="29.513296875" y2="79.80428125" width="0.001" layer="20" curve="119.999997"/>
 </plain>

Commit message: исправил верхнюю плату
Parts:
- moved U$3 89.3 mm to (81.0, 44.0), turned to 60 degrees
- moved U$7 76.7 mm to (81.0, 44.0), flipped to the bottom, turned to 120 degrees
- moved U$2 61.1 mm to (19.0, 44.0), turned to 300 degrees
- moved U$6 5.39 mm to (19.0, 44.0), flipped to the bottom, turned to 240 degrees
- moved U$4 1.00 mm to (50.0, 79.0)
- moved U$8 1.00 mm to (50.0, 79.0)
Routing:
- net SDIO_DAT3: track 75.8 -> 77.3 mm, vias 1 -> 3
- net SDIO_CK: track 46.1 -> 44.8 mm
- net SDIO_DAT1: track 48.5 -> 47.9 mm

Commit message: Почти доделал нижнюю плату
Parts:
- added LED1, LED2: (no value), led:CHIPLED_0603
- added R1, R3: 100R, rcl:R0603
- added U$5, U$9: VIAS-SELECT, NEON-BLADE-2024:VIAS-SELECT
- LIS3MDL: value LIS3MDL-CJMCUБез_отв._зеркальный -> LIS3MDL-CJMCUбез_отв.; device NEON-BLADE-2023:LIS3MDL-CGMSU-NB2023 -> NEON-BLADE-2023:LIS3MDL-CGMSU-NB2023-1
- moved C10 53.0 mm to (74.1, 49.5), turned to 180 degrees
- moved J1 49.2 mm to (22.8, 55.4)
- moved J2 45.0 mm to (68.5, 51.5), turned to 90 degrees
- moved SI2301 42.6 mm to (74.0, 29.0)
- moved C1 41.7 mm to (67.7, 39.0)
- moved R31 40.4 mm to (72.0, 33.4)
- moved R30 39.3 mm to (71.5, 37.5)
- moved BUZZER 32.1 mm to (66.0, 26.5)
- moved R10 9.31 mm to (56.9, 30.7), turned to 90 degrees
- moved R8 8.66 mm to (48.9, 30.7), turned to 90 degrees
- moved R9 3.48 mm to (54.2, 30.7), turned to 90 degrees
- moved C7 3.17 mm to (51.6, 29.2), turned to 180 degrees
- moved R2 1.93 mm to (44.6, 30.8), turned to 90 degrees
- moved R7 1.53 mm to (46.8, 30.8), turned to 90 degrees
- moved AMP 1.00 mm to (47.0, 47.0), turned to 180 degrees
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Connections:
- new net N$10: U$3.6, U$7.6
- new net N$11: U$3.7, U$7.7
- new net N$14: U$3.8, U$7.8
- new net N$15: U$3.9, U$7.9
- new net N$16: LED1.C, U$5.2
- new net N$17: LED1.A, R1.2
- new net N$18: AMP.P$8, R1.1
- new net N$19: LED2.C, U$9.2
- new net N$21: LED2.A, R3.2
- new net N$22: AMP.P$9, R3.1
- new net N$6: U$3.2, U$7.2
- new net N$7: U$3.3, U$7.3
- new net N$8: U$3.4, U$7.4
- new net N$9: U$3.5, U$7.5
- net 5V: now also U$5.3, U$9.3
- net GND: now also U$5.1, U$9.1
Routing:
- net 1MOSI: track 11.0 -> 77.5 mm, vias 0 -> 1
- net 1MISO: track 18.4 -> 83.4 mm, vias 0 -> 1
- net 5V: track 58.5 -> 121.7 mm, vias 1 -> 3
- net 1SCK: track 18.5 -> 53.9 mm, vias 0 -> 1
- net 3V3: track 120.2 -> 154.8 mm, vias 3 -> 1
- net USIL_ON: track 29.1 -> 56.7 mm, vias 0 -> 2
- net CS_LIS: track 0.93 -> 26.0 mm, vias 0 -> 1
- net SDIO_DAT3: track 77.3 -> 55.4 mm, vias 3 -> 1
- net 5MISO: track 0.65 -> 19.2 mm, vias 0 -> 1
- net 5MOSI: track 0.63 -> 16.6 mm, vias 0 -> 1
- net GND: track 215.6 -> 199.8 mm, vias 0 -> 9
- net 5SCK: track 0.62 -> 14.2 mm, vias 0 -> 1
- net SDIO_CMD: track 69.2 -> 56.2 mm, vias 2 -> 1
- net CS_LSM: track 2.09 -> 14.7 mm, vias 0 -> 2
- net CS_NRF: track 0.62 -> 11.9 mm, vias 0 -> 1
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- added copper zone on layer 1, net GND
- added copper zone on layer 16, net GND

Commit message: Проверил плату нижнюю
Parts:
- added U$10: VIAS-SELECT, NEON-BLADE-2024:VIAS-SELECT
- moved C10 6.52 mm to (70.6, 44.0)
- moved R30 2.55 mm to (71.0, 35.0), turned to 0 degrees
- moved R31 1.12 mm to (71.0, 32.9)
- moved NRF24L01P 0.50 mm to (55.1, 68.6)
- moved J1 0.43 mm to (22.8, 55.0)
- moved R7 0.08 mm to (46.8, 30.7)
- moved R2 0.06 mm to (44.6, 30.7)
- turned U$2 to 120 degrees
- turned U$3 to 240 degrees
- turned U$8 to 180 degrees
- renumbered AMP to AMPLIFIRE
Connections:
- removed net N$13: U$8.15
- net 1MISO: now also U$8.13; no longer U$8.3
- net 1MOSI: now also U$8.14; no longer U$8.2
- net 1SCK: now also U$8.15; no longer U$8.1
- net 3V3: now also U$8.11; no longer U$8.5
- net 5MISO: now also U$8.5; no longer U$8.11
- net 5MOSI: now also U$8.6; no longer U$8.10
- net 5SCK: now also U$8.7; no longer U$8.9
- net 5V: now also U$10.3, U$2.9; no longer U$2.1
- net BUZZER: now also U$8.3; no longer U$8.13
- net CE_NRF: now also U$8.9; no longer U$8.7
- net CS_LIS: now also U$8.12; no longer U$8.4
- net CS_LSM: now also U$8.4; no longer U$8.12
- net GND: now also U$10.1, U$8.10; no longer U$8.6
- net N$10: now also U$3.4; no longer U$3.6
- net N$11: now also U$3.3; no longer U$3.7
- net N$12: now also U$3.9, U$7.1; no longer U$8.14
- net N$14: now also U$3.2; no longer U$3.8
- net N$15: now also U$3.1; no longer U$3.9
- net N$2: now also U$8.2
- net N$3: now also U$8.1
- net N$6: now also U$3.8; no longer U$3.2
- net N$7: now also U$3.7; no longer U$3.3
- net N$8: now also U$3.6; no longer U$3.4
- net SCL: now also U$2.1; no longer U$2.9
- net SDA: now also U$2.2; no longer U$2.8
- net SDIO_CMD: now also U$2.6; no longer U$2.4
- net SDIO_DAT0: now also U$2.4; no longer U$2.6
- net SDIO_DAT1: now also U$2.3; no longer U$2.7
- net SDIO_DAT2: now also U$2.8; no longer U$2.2
- net SDIO_DAT3: now also U$2.7; no longer U$2.3
- net USIL_ON: now also U$10.2; no longer U$3.1, U$7.1
Routing:
- net USIL_ON: track 56.7 -> 5.98 mm, vias 2 -> 0
- net GND: track 199.8 -> 235.2 mm, vias 9 -> 10
- net 1SCK: track 53.9 -> 82.9 mm
- net 1MISO: track 83.4 -> 57.4 mm
- net 3V3: track 154.8 -> 145.0 mm, vias 1 -> 9
- net BUZZER: track 57.9 -> 48.9 mm
- net 1MOSI: track 77.5 -> 71.5 mm
- net CS_LIS: track 26.0 -> 20.1 mm
- net SDIO_CMD: track 56.2 -> 52.7 mm
- net 5MISO: track 19.2 -> 16.0 mm
- net CE_NRF: track 9.59 -> 6.81 mm
- net SDIO_DAT2: track 49.3 -> 46.6 mm
- net SDIO_DAT0: track 48.1 -> 45.4 mm
- net N$15: track 2.70 -> 0.00 mm
- net N$7: track 2.70 -> 0.00 mm
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- added copper zone on layer 1, net 3V3
- added copper zone on layer 16, net 3V3
- added copper zone on layer 1, net 5V
Other:
- board text added: "AMP"
- board text added: "ON"

Commit message: Внес поправки
Parts:
- R1, R3: value 100R -> 2k
- moved U$10 2.92 mm to (27.8, 32.5)
- moved NRF24L01P 0.86 mm to (56.0, 68.5)
- renumbered J1 to RADIO, J2 to ANT
Connections:
- removed net NRF_IRQ: NRF24L01P.P$7
- net 3V3: no longer U$1.P$1
- net 5V: now also U$1.P$1
Routing:
- net 5V: track 120.8 -> 142.2 mm
- net 3V3: track 145.0 -> 130.5 mm
- net BUZZER: track 48.9 -> 51.4 mm
- net GND: track 235.2 -> 237.6 mm
- net USIL_ON: track 5.98 -> 4.10 mm
- net CE_NRF: track 6.81 -> 7.39 mm
Other:
- board text added: "3V3"
- board text added: "5V"
- board text added: "APD_FB"
- board text added: "APD_PWM"
- board text added: "BUZZ"
- board text added: "Bottom board [2024] v.1"
- board text added: "CE_RF"
- board text added: "CS_LIS"
- board text added: "CS_LM"
- board text added: "CS_LSM"
- board text added: "CS_NRF"
- board text added: "CS_RF"
- board text added: "CS_TDC"
- board text added: "GND"
- board text added: "MISO"
- board text added: "MOSI"
- board text added: "NEON BLADE"
- board text added: "OFF"
- board text added: "SCK"
- board text added: "SCL"
- board text added: "SDA"
- board text added: "SDIO0"
- board text added: "SDIO1"
- board text added: "SDIO2"
- board text added: "SDIO3"
- board text added: "SD_CK"
- board text added: "SDСMD"
- board text added: "VB"
- board text added: "[NC]"

Commit message: Считаем, что платы готовы к производству
Parts:
- moved LIS3MDL 1.50 mm to (26.6, 66.0)
Routing:
- net 1MOSI: track 71.5 -> 73.3 mm
- net CS_LIS: track 20.1 -> 21.6 mm
- net 1MISO: track 57.4 -> 58.9 mm
- net 3V3: track 130.5 -> 131.7 mm
- net 1SCK: track 82.9 -> 81.7 mm
- net GND: track 237.6 -> 238.8 mm
Changed lines of the file:
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@@
 <attribute name="NAME" x="71.013" y="51.46533125" size="1.2" layer="25" ratio="15" rot="R90" align="center"/>
 </element>
-<element name="LIS3MDL" library="NEON-BLADE-2023" package="LIS3MDL-CGMSU-NB2023-1" value="LIS3MDL-CJMCUбез_отв." x="28.13" y="65.97" smashed="yes" rot="R180">
-<attribute name="NAME" x="31.63" y="73.32" size="1.2" layer="25" ratio="12" rot="R180"/>
+<element name="LIS3MDL" library="NEON-BLADE-2023" package="LIS3MDL-CGMSU-NB2023-1" value="LIS3MDL-CJMCUбез_отв." x="26.63" y="65.97" smashed="yes" rot="R180">
+<attribute name="NAME" x="30.13" y="73.32" size="1.2" layer="25" ratio="12" rot="R180"/>
 </element>
 <element name="LSM6DS3" library="NEON-BLADE-2023" package="LSM6DS3-GY-NB2023" value="LSM6DS3-GY-NB2023" x="74.26" y="65.41" smashed="yes" rot="MR180">
@@
 <wire x1="44.92" y1="76.89360625" x2="44.92" y2="80.35" width="0.5" layer="16"/>
 <wire x1="42.87639375" y1="74.85" x2="37.86" y2="74.85" width="0.5" layer="16"/>
-<wire x1="37.86" y1="74.85" x2="34.48" y2="71.47" width="0.5" layer="16"/>
-<wire x1="34.48" y1="71.47" x2="34.48" y2="69.97" width="0.5" layer="16"/>
-<wire x1="34.48" y1="68.47" x2="25.37" y2="59.36" width="0.3" layer="16"/>
-<wire x1="25.37" y1="59.36" x2="25.37" y2="57.54" width="0.3" layer="16"/>
+<wire x1="37.86" y1="74.85" x2="32.98" y2="69.97" width="0.5" layer="16"/>
+<wire x1="25.37" y1="57.54" x2="25.37" y2="59.86" width="0.3" layer="16"/>
 <wire x1="72.87" y1="56.62" x2="72.87" y2="55.12" width="0.5" layer="1"/>
 <wire x1="72.87" y1="55.12" x2="70.685" y2="52.935" width="0.5" layer="1"/>
 <wire x1="70.685" y1="52.935" x2="68.55" y2="52.935" width="0.5" layer="1"/>
-<wire x1="34.48" y1="68.47" x2="35.475" y2="67.475" width="0.5" layer="16"/>
-<wire x1="34.48" y1="68.47" x2="34.48" y2="69.97" width="0.5" layer="16"/>
+<wire x1="33.13" y1="69.82" x2="32.98" y2="69.97" width="0.5" layer="16"/>
+<wire x1="33.13" y1="69.82" x2="33.13" y2="67.475" width="0.5" layer="16"/>
 <wire x1="76.8" y1="70.41" x2="76.8" y2="68.3" width="0.5" layer="16"/>
 <wire x1="72.87" y1="64.37" x2="72.87" y2="56.62" width="0.5" layer="16"/>
@@
 <wire x1="52.5" y1="30.5" x2="51.65" y2="31.35" width="0.3" layer="16"/>
 <wire x1="51.65" y1="31.35" x2="28.3" y2="31.35" width="0.3" layer="16"/>
-<wire x1="35.475" y1="67.475" x2="38.025" y2="67.475" width="0.5" layer="16"/>
+<wire x1="33.13" y1="67.475" x2="38.025" y2="67.475" width="0.5" layer="16"/>
 <wire x1="38.025" y1="67.475" x2="41.5" y2="64" width="0.5" layer="16"/>
 <wire x1="41.5" y1="64" x2="48.5" y2="64" width="0.5" layer="16"/>
 <wire x1="63.5" y1="40.5" x2="74" y2="30" width="0.5" layer="16"/>
+<wire x1="32.985" y1="67.475" x2="33.13" y2="67.475" width="0.3" layer="16"/>
+<wire x1="25.37" y1="59.86" x2="32.985" y2="67.475" width="0.3" layer="16"/>
 </signal>
 <signal name="3V3">
@@
 <wire x1="50.73" y1="29.25" x2="50.73" y2="29.23" width="0.5" layer="1"/>
 <wire x1="50.73" y1="29.23" x2="50.5" y2="29" width="0.5" layer="1"/>
-<wire x1="37.02" y1="69.97" x2="37.02" y2="71.47" width="0.5" layer="1"/>
-<wire x1="38.555" y1="73.005" x2="37.02" y2="71.47" width="0.5" layer="1"/>
+<wire x1="38.555" y1="73.005" x2="35.52" y2="69.97" width="0.5" layer="1"/>
 <wire x1="38.555" y1="73.005" x2="42.38" y2="73.005" width="0.5" layer="1"/>
 <wire x1="42.38" y1="73.005" x2="47" y2="72.945" width="0.5" layer="1"/>
@@
 <wire x1="38.5" y1="58" x2="37.5" y2="58" width="0.3" layer="16"/>
 <wire x1="36.5" y1="64.5" x2="36.5" y2="58" width="0.3" layer="16"/>
-<wire x1="37.02" y1="69.97" x2="37.02" y2="64.98" width="0.3" layer="1"/>
-<wire x1="37.02" y1="64.98" x2="37.5" y2="64.5" width="0.3" layer="1"/>
+<wire x1="35.52" y1="69.97" x2="35.52" y2="66.48" width="0.3" layer="1"/>
+<wire x1="35.52" y1="66.48" x2="37.5" y2="64.5" width="0.3" layer="1"/>
 <wire x1="44.65" y1="31.55" x2="44.65" y2="32.55" width="0.3" layer="1"/>
 <wire x1="44.65" y1="32.55" x2="36.5" y2="40.7" width="0.3" layer="1"/>
@@
 <via x="39.84" y="80.35" extent="1-16" drill="0.35"/>
 <wire x1="37.574975" y1="80.35" x2="39.84" y2="80.35" width="0.3" layer="1"/>
-<wire x1="24.32" y1="69.97" x2="25.932" y2="71.582" width="0.3" layer="1"/>
+<wire x1="22.82" y1="69.97" x2="24.432" y2="71.582" width="0.3" layer="1"/>
 <wire x1="36.44" y1="78.7971125" x2="36.44" y2="79.215025" width="0.3" layer="1"/>
 <wire x1="36.44" y1="79.215025" x2="37.574975" y2="80.35" width="0.3" layer="1"/>
-<wire x1="25.932" y1="71.582" x2="29.2248875" y2="71.582" width="0.3" layer="1"/>
+<wire x1="24.432" y1="71.582" x2="29.2248875" y2="71.582" width="0.3" layer="1"/>
 <wire x1="29.2248875" y1="71.582" x2="36.44" y2="78.7971125" width="0.3" layer="1"/>
 </signal>
@@
 <wire x1="33.9995" y1="82.9995" x2="32.22" y2="81.22" width="0.3" layer="1"/>
 <wire x1="20.668" y1="69.50939375" x2="20.668" y2="70.43060625" width="0.3" layer="1"/>
-<wire x1="31.94" y1="69.97" x2="30.97260625" y2="69.97" width="0.3" layer="1"/>
-<wire x1="30.97260625" y1="69.97" x2="29.36060625" y2="68.358" width="0.3" layer="1"/>
+<wire x1="30.44" y1="69.97" x2="30.44" y2="69.43739375" width="0.3" layer="1"/>
+<wire x1="30.44" y1="69.43739375" x2="29.36060625" y2="68.358" width="0.3" layer="1"/>
 <wire x1="29.36060625" y1="68.358" x2="21.81939375" y2="68.358" width="0.3" layer="1"/>
 <wire x1="21.81939375" y1="68.358" x2="20.668" y2="69.50939375" width="0.3" layer="1"/>
@@
 <wire x1="34.76" y1="80.35" x2="34.76" y2="77.824225" width="0.3" layer="1"/>
 <wire x1="34.76" y1="77.824225" x2="29.017775" y2="72.082" width="0.3" layer="1"/>
-<wire x1="23.208" y1="70.43060625" x2="23.208" y2="69.50939375" width="0.3" layer="1"/>
-<wire x1="23.208" y1="69.50939375" x2="23.85939375" y2="68.858" width="0.3" layer="1"/>
-<wire x1="29.017775" y1="72.082" x2="24.85939375" y2="72.082" width="0.3" layer="1"/>
-<wire x1="24.85939375" y1="72.082" x2="23.208" y2="70.43060625" width="0.3" layer="1"/>
-<wire x1="27.32060625" y1="68.858" x2="28.43260625" y2="69.97" width="0.3" layer="1"/>
-<wire x1="28.43260625" y1="69.97" x2="29.4" y2="69.97" width="0.3" layer="1"/>
-<wire x1="23.85939375" y1="68.858" x2="27.32060625" y2="68.858" width="0.3" layer="1"/>
+<wire x1="21.708" y1="70.43060625" x2="21.708" y2="69.50939375" width="0.3" layer="1"/>
+<wire x1="21.708" y1="69.50939375" x2="22.35939375" y2="68.858" width="0.3" layer="1"/>
+<wire x1="29.017775" y1="72.082" x2="23.35939375" y2="72.082" width="0.3" layer="1"/>
+<wire x1="23.35939375" y1="72.082" x2="21.708" y2="70.43060625" width="0.3" layer="1"/>
+<wire x1="27.32060625" y1="68.858" x2="27.9" y2="69.43739375" width="0.3" layer="1"/>
+<wire x1="27.9" y1="69.43739375" x2="27.9" y2="69.97" width="0.3" layer="1"/>
+<wire x1="22.35939375" y1="68.858" x2="27.32060625" y2="68.858" width="0.3" layer="1"/>
 </signal>
 <signal name="1MISO">
@@
 <wire x1="36" y1="77.65" x2="29.432" y2="71.082" width="0.3" layer="1"/>
 <wire x1="36" y1="77.65" x2="37.3" y2="77.65" width="0.3" layer="1"/>
-<wire x1="26.86" y1="69.97" x2="27.972" y2="71.082" width="0.3" layer="1"/>
-<wire x1="27.972" y1="71.082" x2="29.432" y2="71.082" width="0.3" layer="1"/>
+<wire x1="25.36" y1="69.97" x2="26.472" y2="71.082" width="0.3" layer="1"/>
+<wire x1="26.472" y1="71.082" x2="29.432" y2="71.082" width="0.3" layer="1"/>
 <wire x1="43.5424875" y1="76.4575125" x2="43.034975" y2="75.95" width="0.3" layer="16"/>
 <wire x1="66.64" y1="76.36" x2="66.64" y2="70.41" width="0.3" layer="16"/>
