File: schematic/board/Down_Main_Board .brd (EAGLE design)
At the start: 79.9 x 73.5 mm, 33 parts

Commit message: теперь точно готовы
Parts:
- moved C10 1.82 mm to (72.1, 45.0)
Routing:
- net GND: track 238.8 -> 242.3 mm, vias 10 -> 12
Other:
- board size 79.9 x 73.5 mm -> 79.8 x 73.5 mm
