File: schematic/board/lidar_made_by_apple.brd (EAGLE design)
At the start: 79.9 x 72.5 mm, 90 parts, among them J1 U.FL-R-SMT-1_10_, J2 U.FL-R-SMT-1_10_

Commit message: переделки по плате
Connections:
- removed net 1MISO: U$17.3
- removed net 1MOSI: U$17.2
- removed net 1SCK: U$17.1
- removed net 5MISO: U$17.11
- removed net 5MOSI: U$17.10
- removed net 5SCK: U$17.9
- removed net CE_NRF: U$17.7
- removed net CS_LIS: U$17.4
- removed net CS_LSM: U$17.12
- removed net CS_NRF: U$17.8
- removed net N$30: U$17.15
- removed net SCL: U$16.9
- removed net SDA: U$16.8
- removed net SDIO_CK: U$16.5
- removed net SDIO_CMD: U$16.4
- removed net SDIO_DAT0: U$16.6
- removed net SDIO_DAT1: U$16.7
- removed net SDIO_DAT2: U$16.2
- removed net SDIO_DAT3: U$16.3
- removed net USIL_ON: U$15.1
- net 3V3: now also L1.1
- net 3V3_REF: no longer L1.1
- net COMP_DAC: now also U$17.13
- net GND: no longer C20.1
- net N$28: now also C20.1; no longer U$17.13
Routing:
- net COMP_DAC: track 0.00 -> 83.2 mm
- net 3V3: track 3.85 -> 43.9 mm, vias 0 -> 2
- net APD_COMP_OUT: track 39.2 -> 42.7 mm
- net GND: track 77.0 -> 79.8 mm
- net N$17: track 24.7 -> 23.3 mm
- net LASER_COMP: track 73.3 -> 74.0 mm

Commit message: ПЕРЕДЕЛАЙ ПАЛТЫ
Parts:
- moved R19 2.81 mm to (64.3, 48.2)
- moved J2 0.60 mm to (67.7, 52.4)
- moved W3 0.60 mm to (67.7, 55.0)
Routing:
- net PGND: track 164.2 -> 158.9 mm
- net I_LASER: track 17.8 -> 20.4 mm
- net V_BAT: track 73.8 -> 74.9 mm
- net N$18: track 3.05 -> 3.65 mm
Other:
- board size 79.9 x 72.5 mm -> 79.9 x 73.5 mm

Commit message: передвинул пинхеадер и поменял значения резисторов
Parts:
- R14: value 20k -> 4k7
- R15: value 1k -> 150
- moved U$15 3.20 mm to (81.0, 44.0)
- moved U$16 3.20 mm to (19.0, 44.0)
Routing:
- net APD_PWM: track 45.4 -> 48.3 mm
- net 4MOSI: track 48.1 -> 51.0 mm
- net APD_FB_VOLT: track 31.9 -> 34.7 mm
- net CS_TDC: track 44.9 -> 47.6 mm
- net 4MISO: track 52.2 -> 54.8 mm
- net 4SCK: track 50.1 -> 52.6 mm
- net 5V: track 41.5 -> 43.8 mm
- net TDC_INT: track 43.5 -> 45.3 mm
- net LASER_COMP: track 74.2 -> 75.8 mm
Changed lines of the file:
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@@
 <attribute name="VALUE" x="33.915" y="42.145" size="1.27" layer="27"/>
 </element>
-<element name="R14" library="rcl" library_urn="urn:adsk.eagle:library:334" package="R0603" package3d_urn="urn:adsk.eagle:package:23555/3" value="20k" x="33.95" y="50" smashed="yes" rot="R90">
+<element name="R14" library="rcl" library_urn="urn:adsk.eagle:library:334" package="R0603" package3d_urn="urn:adsk.eagle:package:23555/3" value="4k7" x="33.95" y="50" smashed="yes" rot="R90">
 <attribute name="NAME" x="33.315" y="49.365" size="1.27" layer="25" rot="R90"/>
 <attribute name="POPULARITY" value="70" x="86.02" y="119.85" size="1.778" layer="27" rot="R90" display="off"/>
@@
 <attribute name="VALUE" x="35.855" y="49.365" size="1.27" layer="27" rot="R90"/>
 </element>
-<element name="R15" library="rcl" library_urn="urn:adsk.eagle:library:334" package="R0603" package3d_urn="urn:adsk.eagle:package:23555/3" value="1k" x="35.35" y="46.9" smashed="yes" rot="R90">
+<element name="R15" library="rcl" library_urn="urn:adsk.eagle:library:334" package="R0603" package3d_urn="urn:adsk.eagle:package:23555/3" value="150" x="35.35" y="46.9" smashed="yes" rot="R90">
 <attribute name="NAME" x="34.715" y="46.265" size="1.27" layer="25" rot="R90"/>
 <attribute name="POPULARITY" value="70" x="92.5" y="63.41" size="1.778" layer="27" rot="R90" display="off"/>
@@
 <attribute name="VALUE" x="52.005" y="60.615" size="1.27" layer="27" rot="R90"/>
 </element>
-<element name="U$15" library="NEON-BLADE-2024" package="PBS_SMD_X9" value="PBS_SMD_X9" x="79" y="41.5" smashed="yes" rot="R60"/>
-<element name="U$16" library="NEON-BLADE-2024" package="PBS_SMD_X9" value="PBS_SMD_X9" x="21" y="41.5" smashed="yes" rot="R300"/>
+<element name="U$15" library="NEON-BLADE-2024" package="PBS_SMD_X9" value="PBS_SMD_X9" x="81" y="44" smashed="yes" rot="R60"/>
+<element name="U$16" library="NEON-BLADE-2024" package="PBS_SMD_X9" value="PBS_SMD_X9" x="19" y="44" smashed="yes" rot="R300"/>
 <element name="U$17" library="NEON-BLADE-2024" package="PBD_SMD_X15" value="PBS_SMD_X15" x="50" y="79" smashed="yes"/>
 </elements>
@@
 <via x="79.3" y="44.5" extent="1-16" drill="0.35"/>
 <wire x1="79.3" y1="44.5" x2="79.963834375" y2="44.5" width="0.2" layer="1"/>
-<wire x1="79.963834375" y1="44.5" x2="81.43913125" y2="43.024703125" width="0.2" layer="1"/>
+<wire x1="79.963834375" y1="44.5" x2="83.43913125" y2="45.524703125" width="0.2" layer="1"/>
 <wire x1="73.63314375" y1="46" x2="74.4132875" y2="46.3867125" width="0.2" layer="1"/>
 </signal>
@@
 <via x="78.2" y="47.8" extent="1-16" drill="0.35"/>
 <wire x1="78.2" y1="47.8" x2="79.145271875" y2="47.8" width="0.2" layer="1"/>
-<wire x1="79.145271875" y1="47.8" x2="80.370865625" y2="46.57440625" width="0.2" layer="1"/>
+<wire x1="79.145271875" y1="47.8" x2="82.370865625" y2="49.07440625" width="0.2" layer="1"/>
 </signal>
 <signal name="N$16">
@@
 <wire x1="71.57384375" y1="23.6" x2="82.981828125" y2="49.06781875" width="0.2" layer="16"/>
 <via x="82.981828125" y="49.06781875" extent="1-16" drill="0.35"/>
-<wire x1="82.981828125" y1="49.06781875" x2="82.910865625" y2="50.973815625" width="0.2" layer="1"/>
+<wire x1="82.981828125" y1="49.06781875" x2="84.910865625" y2="53.473815625" width="0.2" layer="1"/>
 </signal>
 <signal name="N$31">
@@
 <wire x1="75" y1="28.2" x2="79.09456875" y2="35.102275" width="0.2" layer="1"/>
 <wire x1="79.09456875" y1="35.102275" x2="84" y2="44" width="0.2" layer="1"/>
-<wire x1="84" y1="44" x2="83.97913125" y2="47.4241125" width="0.2" layer="1"/>
+<wire x1="84" y1="44" x2="85.97913125" y2="49.9241125" width="0.2" layer="1"/>
 </signal>
 <signal name="N$34">
@@
 <wire x1="29.3796625" y1="55.2836" x2="24.894878125" y2="50.798815625" width="0.5" layer="16"/>
 <contactref element="U$16" pad="1"/>
-<wire x1="17.08913125" y1="50.973815625" x2="24.719878125" y2="50.973815625" width="0.5" layer="1"/>
+<wire x1="15.08913125" y1="53.473815625" x2="24.719878125" y2="50.973815625" width="0.5" layer="1"/>
 <wire x1="24.719878125" y1="50.973815625" x2="24.894878125" y2="50.798815625" width="0.5" layer="1"/>
 <via x="24.894878125" y="50.798815625" extent="1-16" drill="0.35"/>
@@
 <via x="73" y="39" extent="1-16" drill="0.35"/>
 <wire x1="73" y1="39" x2="74.224409375" y2="37.775590625" width="0.2" layer="1"/>
-<wire x1="74.224409375" y1="37.775590625" x2="75.290865625" y2="37.775590625" width="0.2" layer="1"/>
+<wire x1="74.224409375" y1="37.775590625" x2="77.290865625" y2="40.275590625" width="0.2" layer="1"/>
 <wire x1="71.3524" y1="48.445975" x2="71.3524" y2="40.6476" width="0.2" layer="16"/>
 </signal>
@@
 <via x="76" y="39.028121875" extent="1-16" drill="0.35"/>
 <wire x1="76" y1="39.028121875" x2="78.496303125" y2="39.028121875" width="0.2" layer="1"/>
-<wire x1="78.496303125" y1="39.028121875" x2="78.89913125" y2="38.62529375" width="0.2" layer="1"/>
+<wire x1="78.496303125" y1="39.028121875" x2="80.89913125" y2="41.12529375" width="0.2" layer="1"/>
 </signal>
 <signal name="CS_TDC">
@@
 <via x="78" y="44" extent="1-16" drill="0.35"/>
 <wire x1="78" y1="44" x2="78" y2="42.344134375" width="0.2" layer="1"/>
-<wire x1="78" y1="42.344134375" x2="77.830865625" y2="42.175" width="0.2" layer="1"/>
+<wire x1="78" y1="42.344134375" x2="79.830865625" y2="44.675" width="0.2" layer="1"/>
 </signal>
 <signal name="4SCK">
@@
 <via x="75" y="36" extent="1-16" drill="0.35"/>
 <wire x1="75" y1="36" x2="76.35913125" y2="34.64086875" width="0.2" layer="1"/>
-<wire x1="76.35913125" y1="34.64086875" x2="76.35913125" y2="34.225884375" width="0.2" layer="1"/>
+<wire x1="76.35913125" y1="34.64086875" x2="78.35913125" y2="36.725884375" width="0.2" layer="1"/>
 <wire x1="71" y1="48.3" x2="71" y2="40" width="0.2" layer="16"/>
 </signal>

Commit message: чёт сделял
Parts:
- removed R12: 82, rcl:R0603
- removed R32: NC, rcl:R0603
Connections:
- removed net APD_COMP_MCU: R32.2
- removed net N$7: C14.2, R12.1, R13.1
- net 3V3_REF: now also L6.1
- net APD_COMP_OUT: no longer R32.1
- net COMP_DAC: no longer L6.1
- net N$14: now also C14.2, R13.1; no longer R12.2
Routing:
- net COMP_DAC: track 83.2 -> 0.00 mm
- net 3V3_REF: track 70.4 -> 80.9 mm
- net N$14: track 2.25 -> 8.18 mm
- net N$7: track 4.22 -> 0.00 mm
- net APD_COMP_OUT: track 42.7 -> 38.7 mm
- net CS_TDC: track 47.6 -> 45.5 mm
- net APD_PWM: track 48.3 -> 49.7 mm
- net V_BAT: track 74.9 -> 75.7 mm
- net 4SCK: track 52.6 -> 51.8 mm

Commit message: опять чёт сделял
Connections:
- removed net COMP_DAC: U$17.13
Routing:
- net APD_COMP_OUT: track 38.7 -> 42.7 mm
Changed lines of the file:
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@@
 <wire x1="31.8" y1="41.6" x2="32" y2="41.8" width="0.2" layer="1"/>
-</signal>
-<signal name="COMP_DAC">
-<contactref element="U$17" pad="13"/>
 </signal>
 <signal name="N$15">
@@
 <wire x1="29.8" y1="52.6" x2="31.9812" y2="54.7812" width="0.2" layer="16"/>
 <via x="29.8" y="52.6" extent="1-16" drill="0.35"/>
-<wire x1="29.8" y1="52.6" x2="29.82" y2="52.58" width="0.2" layer="1"/>
 <wire x1="43.2694" y1="57.2694" x2="43.2694" y2="63.2506" width="0.2" layer="16"/>
 <wire x1="31.9812" y1="54.7812" x2="40.7812" y2="54.7812" width="0.2" layer="16"/>
@@
 <wire x1="44.2694" y1="64.2506" x2="43.2694" y2="63.2506" width="0.2" layer="16"/>
 <wire x1="44.2694" y1="72.2506" x2="44.2694" y2="64.2506" width="0.2" layer="16"/>
-<wire x1="29.82" y1="48.5" x2="29.82" y2="52.58" width="0" layer="19" extent="1-1"/>
+<wire x1="29.8" y1="52.6" x2="29.82" y2="52.58" width="0.2" layer="1"/>
+<wire x1="29.82" y1="52.58" x2="29.82" y2="48.5" width="0.2" layer="1"/>
 </signal>
 <signal name="N$18">

Commit message: поправил контур всех плат
Connections:
- net N$18: now also J2.2
- net PGND: no longer J2.2
Routing:
- net N$18: track 3.65 -> 6.79 mm
Changed lines of the file:
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@@
 <wire x1="10.0594" y1="52.179140625" x2="25.751290625" y2="25" width="0.001" layer="20"/>
 <wire x1="34.98128125" y1="25" x2="25.751290625" y2="25" width="0.001" layer="20"/>
-<wire x1="75.794009375" y1="75.35091875" x2="79.71443125" y2="76.777840625" width="0.001" layer="20"/>
+<wire x1="75.794" y1="75.3509" x2="79.71443125" y2="76.777840625" width="0.001" layer="20"/>
 <wire x1="68.44266875" y1="14.94365" x2="65.56791875" y2="17.355859375" width="0.001" layer="20"/>
-<wire x1="28.86165" y1="83.5" x2="29.5133" y2="79.80428125" width="0.001" layer="20"/>
+<wire x1="28.86165" y1="83.5" x2="29.513296875" y2="79.80428125" width="0.001" layer="20"/>
 <wire x1="39.90531875" y1="20.868240625" x2="41.66693125" y2="10.87763125" width="0.001" layer="20"/>
 <wire x1="71.13835" y1="83.5" x2="70.4867" y2="79.80428125" width="0.001" layer="20"/>
-<wire x1="59.05753125" y1="14.98626875" x2="58.33306875" y2="10.87763125" width="0.001" layer="20"/>
+<wire x1="59.0575" y1="14.98626875" x2="58.33306875" y2="10.87763125" width="0.001" layer="20"/>
 <wire x1="20.28556875" y1="76.777840625" x2="24.205990625" y2="75.35091875" width="0.001" layer="20"/>
 <wire x1="68.44266875" y1="14.94365" x2="89.9406" y2="52.179140625" width="0.001" layer="20"/>
@@
 <wire x1="89.9406" y1="52.179140625" x2="79.71443125" y2="76.777840625" width="0.001" layer="20" curve="38.901385"/>
 <wire x1="20.28556875" y1="76.777840625" x2="10.0594" y2="52.179140625" width="0.001" layer="20" curve="38.901385"/>
-<wire x1="39.90531875" y1="20.868240625" x2="34.98128125" y2="25.000003125" width="0.001" layer="20" curve="79.999971"/>
+<wire x1="39.90531875" y1="20.868240625" x2="34.98128125" y2="25" width="0.001" layer="20" curve="79.999971"/>
 <wire x1="24.205990625" y1="75.35091875" x2="29.513296875" y2="79.80428125" width="0.001" layer="20" curve="119.999997"/>
-<wire x1="70.4867" y1="79.80428125" x2="75.79400625" y2="75.350921875" width="0.001" layer="20" curve="120.000013"/>
-<wire x1="65.56791875" y1="17.355859375" x2="59.057534375" y2="14.98626875" width="0.001" layer="20" curve="120.000001"/>
+<wire x1="70.4867" y1="79.80428125" x2="75.794" y2="75.3509" width="0.001" layer="20" curve="120.000013"/>
+<wire x1="65.56791875" y1="17.355859375" x2="59.0575" y2="14.98626875" width="0.001" layer="20" curve="120.000001"/>
 <circle x="37.5" y="52" radius="1.15" width="0.001" layer="20"/>
 <circle x="27.5" y="42" radius="1.15" width="0.001" layer="20"/>
@@
 <contactref element="W3" pad="1"/>
 <contactref element="W1" pad="P$1"/>
-<contactref element="J2" pad="2"/>
 <contactref element="C2" pad="1"/>
 <contactref element="U$11" pad="GND"/>
@@
 <wire x1="78.3424" y1="66.6576" x2="80.2876" y2="64.7124" width="0.5" layer="1"/>
 <wire x1="76.26908125" y1="70.9" x2="78.3424" y2="68.82668125" width="0.5" layer="1"/>
-<wire x1="66.175" y1="52.39" x2="66.175" y2="54.045" width="0.5" layer="1"/>
-<wire x1="66.175" y1="54.045" x2="67.15" y2="55.02" width="0.5" layer="1"/>
 <wire x1="63.25" y1="57.5" x2="63.25" y2="59.6" width="0.5" layer="1"/>
 <wire x1="63.25" y1="59.6" x2="60" y2="62.85" width="0.5" layer="1"/>
@@
 <wire x1="80.7476" y1="57.7476" x2="75.2024" y2="52.2024" width="0.5" layer="1"/>
 <wire x1="70.8264" y1="43.9037625" x2="70.8264" y2="41.56241875" width="0.5" layer="1"/>
-<wire x1="76.78455" y1="58.9276" x2="75.7276" y2="58.9276" width="0.2" layer="1"/>
 <wire x1="78.41" y1="60.71" x2="77.0124" y2="59.3124" width="0.2" layer="1"/>
 <wire x1="77.0124" y1="59.3124" x2="77.0124" y2="59.15545" width="0.2" layer="1"/>
 <wire x1="77.0124" y1="59.15545" x2="76.78455" y2="58.9276" width="0.2" layer="1"/>
-<wire x1="75.7276" y1="58.9276" x2="64.6776" y2="58.9276" width="0.2" layer="1"/>
+<wire x1="76.78455" y1="58.9276" x2="64.6776" y2="58.9276" width="0.2" layer="1"/>
 <wire x1="64.6776" y1="58.9276" x2="63.25" y2="57.5" width="0.2" layer="1"/>
 <wire x1="69.89455" y1="75.2024" x2="68.58545" y2="75.2024" width="0.2" layer="1"/>
@@
 <wire x1="70.8424" y1="72.5576" x2="70.8424" y2="74.25455" width="0.2" layer="1"/>
 <wire x1="70.8424" y1="74.25455" x2="69.89455" y2="75.2024" width="0.2" layer="1"/>
-<wire x1="64.35" y1="49.05" x2="64.35" y2="50.565" width="0.5" layer="1"/>
-<wire x1="64.35" y1="50.565" x2="66.175" y2="52.39" width="0.5" layer="1"/>
 <wire x1="67.15" y1="55.02" x2="65.4724" y2="56.6976" width="0.2" layer="1"/>
 <wire x1="65.4724" y1="56.6976" x2="64.34545" y2="56.6976" width="0.2" layer="1"/>
 <wire x1="63.54305" y1="57.5" x2="63.25" y2="57.5" width="0.2" layer="1"/>
 <wire x1="64.34545" y1="56.6976" x2="63.54305" y2="57.5" width="0.2" layer="1"/>
+<wire x1="65.48331875" y1="53.8924" x2="66.0224" y2="53.8924" width="0.5" layer="1"/>
+<wire x1="64.35" y1="52.75908125" x2="65.48331875" y2="53.8924" width="0.5" layer="1"/>
+<wire x1="64.35" y1="49.05" x2="64.35" y2="52.75908125" width="0.5" layer="1"/>
+<wire x1="66.0224" y1="53.8924" x2="67.15" y2="55.02" width="0.5" layer="1"/>
 </signal>
 <signal name="LASER_PULSE">
@@
 <contactref element="J2" pad="1"/>
 <contactref element="W3" pad="2"/>
-<wire x1="69.15" y1="54.02" x2="69.15" y2="51.815" width="0.5" layer="1"/>
+<wire x1="69.15" y1="54.02" x2="69.15" y2="52" width="0.5" layer="1"/>
+<wire x1="69.15" y1="52" x2="69.15" y2="51.815" width="0.5" layer="1"/>
 <wire x1="69.125" y1="52.39" x2="69.15" y2="52.415" width="0.5" layer="1"/>
 <wire x1="69.15" y1="54.02" x2="68.15" y2="55.02" width="0.5" layer="1"/>
+<contactref element="J2" pad="2"/>
+<wire x1="66.175" y1="52.39" x2="68.76" y2="52.39" width="0.5" layer="1"/>
+<wire x1="68.76" y1="52.39" x2="69.15" y2="52" width="0.5" layer="1"/>
+<wire x1="69.15" y1="51.815" x2="69.125" y2="52.39" width="0" layer="19" extent="1-1"/>
 </signal>
 <signal name="N$20">

Commit message: Ошибка повторенная дважды называется - выбор
Parts:
- moved C8 47.0 mm to (54.0, 71.0), turned to 0 degrees
- moved C21 45.1 mm to (61.8, 28.7)
- moved C29 45.1 mm to (61.3, 25.7)
- moved C3 45.1 mm to (47.4, 16.2)
- moved C7 45.1 mm to (52.6, 16.2)
- moved R24 45.1 mm to (58.9, 29.8)
- moved R31 45.1 mm to (59.2, 25.7)
- moved R4 45.1 mm to (50.0, 17.1)
- moved U$10 45.1 mm to (51.5, 28.3)
- moved U$9 45.1 mm to (56.4, 29.8)
- moved U$14 45.1 mm to (50.0, 21.6)
- moved C18 45.0 mm to (44.0, 29.0)
- moved C20 45.0 mm to (44.0, 25.8)
- moved L9 45.0 mm to (44.0, 32.0)
- moved C22 45.0 mm to (61.8, 30.9)
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Connections:
- removed net N$28: C20.1
- net GND: now also C20.1
- net LASER_COMP: no longer U$15.6
Routing:
- net V_BAT: track 75.7 -> 16.2 mm, vias 2 -> 0
- net LASER_COMP: track 75.7 -> 28.3 mm, vias 5 -> 2
- net GND: track 79.8 -> 124.4 mm, vias 3 -> 9
- net PGND: track 159.3 -> 119.6 mm, vias 0 -> 11
- net APD_COMP_OUT: track 42.7 -> 76.6 mm
- net 3V3: track 44.0 -> 75.9 mm
- net 3V3_REF: track 80.9 -> 53.9 mm
- net I_LASER: track 20.4 -> 46.9 mm, vias 0 -> 2
- net APD_PWM: track 49.7 -> 25.8 mm
- net 4SCK: track 51.8 -> 35.7 mm, vias 2 -> 0
- net N$12: track 4.15 -> 19.5 mm, vias 0 -> 2
- net N$17: track 23.3 -> 8.35 mm
- net APD_V: track 23.2 -> 38.0 mm, vias 0 -> 2
- net N$13: track 19.8 -> 5.17 mm
- net VLASER: track 8.81 -> 23.0 mm
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