File: schematic/board/lidar_made_by_apple.brd (EAGLE design)
At the start: 79.9 x 73.5 mm, 88 parts, among them J1 U.FL-R-SMT-1_10_, J2 U.FL-R-SMT-1_10_

Commit message: добавил полигоны на плату и добавил буквы на разъём
Parts:
- moved W3 34.5 mm to (61.0, 34.2), turned to 270 degrees
- moved J2 34.4 mm to (57.7, 35.9), turned to 0 degrees
- moved R20 25.2 mm to (57.7, 41.2), turned to 90 degrees
- moved C11 17.7 mm to (43.3, 69.4)
- moved R10 17.7 mm to (43.3, 71.5)
- moved R19 17.5 mm to (50.5, 46.0)
- moved J1 17.3 mm to (21.0, 57.5), turned to 180 degrees
- moved D1 17.1 mm to (46.2, 71.5), turned to 270 degrees
- moved L5 15.5 mm to (50.4, 71.5), turned to 180 degrees
- moved C10 15.3 mm to (46.4, 73.6), turned to 270 degrees
- moved L4 14.6 mm to (54.0, 73.8)
- moved C19 14.3 mm to (48.2, 57.1)
- moved U$12 14.0 mm to (43.0, 36.5)
- moved R8 13.9 mm to (46.4, 69.4), turned to 90 degrees
- moved U$13 13.6 mm to (52.5, 67.5), turned to 90 degrees
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Routing:
- net APD_V: track 38.0 -> 77.8 mm, vias 4 -> 2
- net AGND: track 137.2 -> 111.8 mm, vias 17 -> 34
- net V_BAT: track 16.2 -> 36.4 mm
- net 3V3: track 33.0 -> 49.9 mm
- net GND: track 86.3 -> 69.9 mm, vias 6 -> 9
- net I_LASER: track 50.0 -> 35.0 mm
- net APD_COMP_OUT: track 79.3 -> 65.2 mm
- net 3V3_REF: track 72.2 -> 58.6 mm, vias 2 -> 0
- net PGND: track 136.6 -> 123.2 mm, vias 11 -> 25
- net APD_FB_VOLT: track 44.0 -> 54.0 mm
- net N$32: track 13.6 -> 4.60 mm
- net N$26: track 13.4 -> 5.00 mm
- net APD_PWM: track 25.8 -> 32.9 mm
- net CS_TDC: track 37.0 -> 43.9 mm, vias 2 -> 0
- net V_TDC: track 48.3 -> 43.5 mm, vias 5 -> 4
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- added copper zone on layer 1, net N$21
- added copper zone on layer 1, net N$26
- added copper zone on layer 1, net N$31
- added copper zone on layer 1, net N$36
Other:
- outline, holes or cut-outs redrawn
- board text added: "3V3"
- board text added: "5V"
- board text added: "APD"
- board text added: "CE_NRF"
- board text added: "CS_LIS"
- board text added: "CS_LSM"
- board text added: "CS_NRF"
- board text added: "CS_T"
- board text added: "GND"
- board text added: "Laser"
- board text added: "MISO"
- board text added: "MOSI"
- board text added: "SCK"
- board text added: "SCL"
- board text added: "SD.СMD"
- board text added: "SDA"
- board text added: "SDIO0"
- board text added: "SDIO1"
- board text added: "SDIO2"
- board text added: "SDIO3"
- board text added: "SD_CK"
- board text added: "T_INT"
- board text added: "U_ON"
- board text added: "V_BAT"

Commit message: забыи отладочные пины...
Parts:
- C18: value 22F -> 22uF
- C19, C2, C9: device rcl:C1210 -> rcl:C1206
Connections:
- net TDC_INT: no longer U$15.7
Routing:
- net TDC_INT: track 49.8 -> 0.00 mm, vias 2 -> 0
- net VLASER: track 19.6 -> 17.6 mm
- net N$6: track 7.06 -> 5.16 mm

Commit message: Убрал дырку и 100501 раз изменил плату лидара
Parts:
- added U$18, U$19: (no value), NEON-BLADE-2024:VIAS-CONNECT
- C10, C11: value 10nF -> 10nF 250v
- C16, C18, C20: device rcl:C1210 -> rcl:C1206
- C17: value 20nF -> 20nF low esr
- R2: value 47 -> 100R
- moved VR1 5.95 mm to (73.7, 51.2)
- moved C9 5.81 mm to (65.3, 56.6), turned to 0 degrees
- moved U$11 5.69 mm to (73.0, 56.3)
- moved R5 5.19 mm to (68.6, 53.8)
- moved C2 4.31 mm to (78.1, 56.0), turned to 180 degrees
- moved D2 3.63 mm to (68.1, 58.6), turned to 270 degrees
- moved L3 3.07 mm to (73.0, 62.6)
- moved L2 1.39 mm to (77.2, 64.3)
Connections:
- new net APD_V_: R1.2, U$18.2
- new net VLASER_: L8.1, R18.2, U$19.2
- net APD_V: now also U$18.1; no longer R1.2
- net VLASER: now also U$19.1; no longer L8.1, R18.2
Routing:
- net APD_V: track 77.8 -> 5.09 mm, vias 2 -> 0
- net APD_V_: track 0.00 -> 71.7 mm, vias 0 -> 2
- net PGND: track 122.8 -> 132.1 mm
- net VLASER: track 17.6 -> 10.1 mm
- net VLASER_: track 0.00 -> 7.46 mm
- net V_BAT: track 36.4 -> 31.8 mm
- net N$26: track 5.00 -> 9.12 mm
- net N$21: track 10.9 -> 14.9 mm
- net N$33: track 8.75 -> 7.04 mm
- net GND: track 69.9 -> 68.4 mm
- net N$27: track 5.48 -> 4.18 mm
- net V_TDC: track 43.5 -> 42.9 mm
- net N$6: track 5.16 -> 4.60 mm
Other:
- board text added: "APD_V"
- board text added: "V_laser"

Commit message: Считаем, что платы готовы к производству
Parts:
- C10, C33: device rcl:C0603 -> rcl:C0805
- C11: value 10nF 250v -> 10nF 250V; device rcl:C0603 -> rcl:C0805
- C15, C29: value 100nf -> 100nF
- C17: value 20nF low esr -> 22nF low ESR
- C8: value 100pf -> 100pF
- L3: value L_10MKH -> 10uH
- R15: value 150 -> 150R
- R19: value 0.1 -> R100; device rcl:R0603 -> rcl:R2512
- R20, R7: value 47 -> 47R
- R27: value 0 -> 0R
- moved R19 17.6 mm to (65.7, 37.2), turned to 60 degrees
- moved U$19 6.69 mm to (61.9, 60.1)
- moved C17 5.46 mm to (58.0, 49.9), turned to 180 degrees
- moved C11 5.41 mm to (38.8, 72.4), turned to 270 degrees
- moved L9 5.30 mm to (45.5, 34.3)
- moved C2 5.12 mm to (73.0, 56.4), turned to 0 degrees
- moved R9 4.71 mm to (44.4, 68.3), turned to 270 degrees
- moved R8 4.24 mm to (42.3, 68.3)
- moved R2 3.54 mm to (55.4, 68.2), turned to 90 degrees
- moved R3 3.47 mm to (53.2, 68.2), turned to 270 degrees
- moved U$18 3.26 mm to (36.6, 71.5)
- moved C8 3.16 mm to (46.5, 68.3), turned to 270 degrees
- moved U$11 2.90 mm to (72.9, 59.2)
- moved C9 2.66 mm to (66.8, 58.8), turned to 90 degrees
- moved U$3 2.66 mm to (61.9, 45.0)
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- renumbered U$12 to REF3033
Connections:
- removed net N$34: C8.1, R9.1
- removed net TDC_INT: U$10.8
- net PGND: now also C8.1, R9.1
Routing:
- net PGND: track 132.1 -> 149.7 mm, vias 25 -> 37
- net APD_PWM: track 32.9 -> 40.6 mm
- net N$21: track 14.9 -> 7.55 mm
- net N$26: track 9.12 -> 1.80 mm
- net VLASER: track 10.1 -> 17.2 mm
- net N$27: track 4.18 -> 11.2 mm
- net N$35: track 9.60 -> 2.76 mm
- net GND: track 68.4 -> 63.3 mm, vias 9 -> 10
- net 3V3_REF: track 58.6 -> 54.0 mm
- net N$33: track 7.04 -> 2.80 mm
- net V_TDC: track 42.9 -> 46.9 mm
- net N$32: track 4.60 -> 7.51 mm
- net N$18: track 6.97 -> 4.38 mm
- net APD_FB_VOLT: track 54.0 -> 56.1 mm
- net N$34: track 2.05 -> 0.00 mm
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- added copper zone on layer 1, net APD_V
- added copper zone on layer 1, net N$32
- added copper zone on layer 1, net VLASER
- added copper zone on layer 1, net V_BAT
Other:
- board text added: "ADCMP600"
- board text added: "APD_FB"
- board text added: "APD_PWM"
- board text added: "BASS2-02"
- board text added: "BAV99"
- board text added: "BSS131"
- board text added: "BSZ165N04NS-G"
- board text added: "BUZZ"
- board text added: "C005R 32kHz"
- board text added: "CE_RF"
- board text added: "CS_TDC"
- board text added: "HC49S 4 MHz"
- board text added: "LIDAR board [2024] v.1"
- board text added: "MAPD-07-013"
- board text added: "MAX40658"
- board text added: "NEON BLADE"
- board text added: "SDСMD"
- board text added: "SPL-PL-90_3"
- board text added: "TDC-GP21"
- board text added: "UCC27511"
- board text added: "VB"
- board text added: "[NC]"
- board text removed: "CE_NRF"
- board text removed: "CS_T"
- board text removed: "SD.СMD"
- board text removed: "T_INT"
- board text removed: "U_ON"
- board text removed: "V_BAT"

Commit message: теперь точно готовы
Parts:
- moved C3 0.30 mm to (47.4, 17.4)
- moved C7 0.30 mm to (52.6, 17.4)
- moved R4 0.30 mm to (50.0, 17.9)
- moved C10 0.10 mm to (44.1, 72.5)
- moved C11 0.10 mm to (38.8, 72.5)
- moved U$18 0.10 mm to (36.6, 71.6)
Routing:
- net AGND: track 110.7 -> 137.8 mm
- net GND: track 63.3 -> 69.5 mm
- net N$26: track 1.80 -> 3.72 mm
- net N$32: track 7.51 -> 5.69 mm
Other:
- board size 79.9 x 73.5 mm -> 79.8 x 73.5 mm

Commit message: переделал плату лидара(((((
Parts:
- removed U$1: UCC27511DBVR, NEON-BLADE-2024:UCC27511DBVR
- added U$12: LM5114, NEON-BLADE-2024:SOT23-6
- L3: device NEON-BLADE-2024:L_1210 -> NEON-BLADE-2024:L_12X12
- moved L2 9.51 mm to (71.9, 72.2)
- moved L3 6.51 mm to (68.5, 67.3)
- moved C9 1.70 mm to (65.1, 58.7)
- moved D2 1.51 mm to (67.8, 60.0)
- moved R26 1.10 mm to (45.9, 47.3)
- moved R27 1.10 mm to (42.7, 47.3)
- moved C14 0.60 mm to (34.6, 56.2)
- moved L6 0.60 mm to (34.6, 59.4)
- moved L7 0.60 mm to (32.5, 59.4)
- moved R13 0.60 mm to (32.5, 56.2)
- moved C15 0.50 mm to (29.1, 60.4)
- moved C23 0.50 mm to (44.6, 54.5)
- moved R14 0.50 mm to (25.7, 56.2)
- moved R17 0.50 mm to (25.7, 59.4)
- moved R23 0.50 mm to (41.5, 54.5)
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Connections:
- net LASER_PULSE: now also U$12.6; no longer U$1.P$6
- net N$1: now also U$12.2, U$12.3; no longer U$1.P$2, U$1.P$3
- net N$2: now also U$12.1; no longer U$1.P$1
- net N$21: now also L3.P$1; no longer L3.1
- net N$26: now also L3.P$2; no longer L3.2
- net PGND: now also U$12.4, U$12.5; no longer U$1.P$4, U$1.P$5
Routing:
- net V_BAT: track 30.6 -> 20.5 mm
- net N$21: track 7.55 -> 16.2 mm
- net PGND: track 149.7 -> 156.0 mm, vias 37 -> 38
- net AGND: track 137.8 -> 141.2 mm
- net VLASER: track 17.2 -> 15.7 mm
- net N$1: track 12.8 -> 13.9 mm
- net LASER_COMP: track 29.8 -> 28.7 mm
- net N$26: track 3.72 -> 2.75 mm
- net LASER_PULSE: track 39.8 -> 39.0 mm
- net COMP_P: track 5.78 -> 6.55 mm
- net COMP_N: track 5.68 -> 6.44 mm
- net 3V3_REF: track 54.0 -> 53.3 mm
- net N$17: track 3.62 -> 4.28 mm
- net N$15: track 3.48 -> 4.02 mm
Other:
- board text added: "LM5114"
- board text removed: "UCC27511"

Commit message: ещё раз(((((((((((((((((((((((((((((((((((((
Parts:
- moved C5 0.30 mm to (32.6, 49.9)
Connections:
- net AGND: now also U$5.P$8, U$5.P$9
- net N$3: now also U$2.P$9
Routing:
- net N$11: track 13.6 -> 21.1 mm
- net N$3: track 7.75 -> 14.4 mm
- net PGND: track 156.0 -> 158.6 mm
- net N$1: track 13.9 -> 16.2 mm, vias 0 -> 1
- net N$10: track 5.91 -> 7.37 mm
- net AGND: track 141.2 -> 142.4 mm, vias 34 -> 35

Commit message: этого ни кто не видел
Parts:
- moved L2 5.32 mm to (77.2, 71.8)
- moved C9 0.20 mm to (65.1, 58.5)
Routing:
- net V_BAT: track 20.5 -> 26.4 mm
Changed lines of the file:
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@@
 <text x="19.4" y="59.9" size="1.2" layer="25" ratio="15">APD</text>
 <text x="34.9" y="69.4" size="0.8" layer="25" ratio="15">APD_V</text>
-<text x="60" y="61.5" size="0.8" layer="25" ratio="15">V_laser</text>
+<text x="58" y="61.2" size="0.8" layer="25" ratio="15">V_laser</text>
 <text x="29.1" y="44.4" size="0.8" layer="25" ratio="15">MAX40658</text>
 <text x="26.4" y="62.1" size="0.8" layer="25" ratio="15">ADCMP600</text>
@@
 <attribute name="VALUE" x="69.805" y="69.875" size="0.8" layer="27" ratio="15" rot="R180"/>
 </element>
-<element name="L2" library="NEON-BLADE-2024" package="L_BEAD" value="L_BEAD" x="71.9" y="72.2" smashed="yes" rot="R90">
-<attribute name="VALUE" x="73.505" y="70.265" size="0.8" layer="27" ratio="15" rot="R90"/>
+<element name="L2" library="NEON-BLADE-2024" package="L_BEAD" value="L_BEAD" x="77.2" y="71.8" smashed="yes" rot="R90">
+<attribute name="VALUE" x="78.805" y="69.865" size="0.8" layer="27" ratio="15" rot="R90"/>
 </element>
 <element name="C2" library="rcl" library_urn="urn:adsk.eagle:library:334" package="C1206" package3d_urn="urn:adsk.eagle:package:23618/2" value="10uF" x="73" y="56.4" smashed="yes">
@@
 <attribute name="VALUE" x="70.375" y="55.095" size="0.8" layer="27" ratio="15" rot="R90"/>
 </element>
-<element name="C9" library="rcl" library_urn="urn:adsk.eagle:library:334" package="C1206" package3d_urn="urn:adsk.eagle:package:23618/2" value="10uF" x="65.1" y="58.7" smashed="yes" rot="R90">
-<attribute name="POPULARITY" value="54" x="141.6" y="35.7" size="1.778" layer="27" rot="R90" display="off"/>
-<attribute name="SPICEPREFIX" value="C" x="141.6" y="35.7" size="1.778" layer="27" rot="R90" display="off"/>
-<attribute name="VALUE" x="63.975" y="57.395" size="0.8" layer="27" ratio="15" rot="R90"/>
+<element name="C9" library="rcl" library_urn="urn:adsk.eagle:library:334" package="C1206" package3d_urn="urn:adsk.eagle:package:23618/2" value="10uF" x="65.1" y="58.5" smashed="yes" rot="R90">
+<attribute name="POPULARITY" value="54" x="141.6" y="35.5" size="1.778" layer="27" rot="R90" display="off"/>
+<attribute name="SPICEPREFIX" value="C" x="141.6" y="35.5" size="1.778" layer="27" rot="R90" display="off"/>
+<attribute name="VALUE" x="63.975" y="57.195" size="0.8" layer="27" ratio="15" rot="R90"/>
 </element>
 <element name="VR1" library="NEON-BLADE-2024" package="TRIM_3362P-1-502LF" value="3362P-1-502LF" x="73.6" y="51.1" smashed="yes" rot="R180">
@@
 <wire x1="70.3" y1="56.4" x2="71.6" y2="56.4" width="0.2" layer="1"/>
 <wire x1="71.1" y1="59.23" x2="70.3" y2="59.23" width="0.2" layer="1"/>
-<wire x1="68.8657375" y1="57.3" x2="65.1" y2="57.3" width="0.2" layer="1"/>
+<wire x1="68.8657375" y1="57.3" x2="68.6657375" y2="57.1" width="0.2" layer="1"/>
+<wire x1="68.6657375" y1="57.1" x2="65.1" y2="57.1" width="0.2" layer="1"/>
 <wire x1="68.8657375" y1="57.3" x2="70.3" y2="58.7342625" width="0.2" layer="1"/>
 <wire x1="69.7657375" y1="56.4" x2="68.8657375" y2="57.3" width="0.2" layer="16"/>
@@
 <wire x1="64.9" y1="54.25" x2="62.4" y2="56.75" width="0.5" layer="1"/>
 <wire x1="62.4" y1="56.75" x2="62.4" y2="60.1" width="0.5" layer="1"/>
-<wire x1="67.13" y1="60" x2="67.03" y2="60.1" width="0.2" layer="1"/>
-<wire x1="67.03" y1="60.1" x2="65.1" y2="60.1" width="0.2" layer="1"/>
-<wire x1="65.1" y1="60.1" x2="62.4" y2="60.1" width="0.5" layer="1"/>
+<wire x1="67.13" y1="60" x2="67.03" y2="59.9" width="0.2" layer="1"/>
+<wire x1="67.03" y1="59.9" x2="65.1" y2="59.9" width="0.2" layer="1"/>
+<wire x1="65.1" y1="59.9" x2="62.6" y2="59.9" width="0.5" layer="1"/>
+<wire x1="62.6" y1="59.9" x2="62.4" y2="60.1" width="0.5" layer="1"/>
 <polygon width="0.2" layer="1" thermals="no">
 <vertex x="67.8" y="62.2"/>
@@
 <wire x1="74.7" y1="56.7" x2="74.7" y2="58.28" width="0.2" layer="1"/>
 <wire x1="74.7" y1="58.28" x2="74.7" y2="60.18" width="0.2" layer="1"/>
-<wire x1="71.9" y1="71.35" x2="73.55" y2="69.7" width="0.2" layer="1"/>
-<wire x1="73.55" y1="69.7" x2="73.55" y2="67.3" width="0.2" layer="1"/>
+<wire x1="77.2" y1="70.95" x2="73.55" y2="67.3" width="0.2" layer="1"/>
 <wire x1="73.55" y1="67.3" x2="74.7" y2="66.15" width="0.2" layer="1"/>
 <wire x1="74.7" y1="66.15" x2="74.7" y2="60.18" width="0.2" layer="1"/>
@@
 <wire x1="63.24" y1="77.65" x2="58.59" y2="73" width="0.5" layer="1"/>
 <wire x1="58.59" y1="73" x2="55.85" y2="73" width="0.5" layer="1"/>
-<wire x1="71.9" y1="73.05" x2="71.9" y2="74.15" width="0.5" layer="1"/>
-<wire x1="65.24" y1="77.65" x2="68.4" y2="77.65" width="0.5" layer="1"/>
-<wire x1="71.9" y1="74.15" x2="68.4" y2="77.65" width="0.5" layer="1"/>
+<wire x1="68.5" y1="72.65" x2="65.24" y2="75.91" width="0.5" layer="1"/>
+<wire x1="65.24" y1="77.65" x2="65.24" y2="75.91" width="0.5" layer="1"/>
+<wire x1="77.2" y1="72.65" x2="68.5" y2="72.65" width="0.5" layer="1"/>
 <polygon width="0.2" layer="1" rank="2">
 <vertex x="60.9" y="79.1"/>
